File: page_2.kicad_sch (KiCad schematic)
At the start: 75 parts, among them J201 Conn_01x05, J601 USB_C_Receptacle_USB2.0_16P, J901 Micro_SD_Card_Det_Hirose_DM3AT, SW201 BOOT, SW202 RESET, T201 TP 201, U202 TCA9535PWR, U203 TPS3840DL42DBVR, U401 W25N01GVZEIG, U601 USBLC6-2SC6, U602 USBLC6-2SC6, U702 ATECC608B-SSHDA, U801 ASM330LHHTR, U802 TMP1075DGKR, U901 TPS22918TDBVTQ1, U902 SN74AXC4T245QPWRQ1, U903 SN74AXC4T245QPWRQ1

Commit message: More adjustment
Parts:
- renumbered D2 to D201
Changed lines of the file:
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@@
 		(in_pos_files yes)
 		(dnp no)
-		(property "Reference" "D2"
+		(property "Reference" "D201"
 			(at 453.898 128.524 0)
 			(show_name no)
@@
 			(project "Tracker"
 				(path "/d199d368-1586-417b-b5ba-1502c361dff2"
-					(reference "D2")
+					(reference "D201")
 					(unit 1)
 				)

Commit message: dec
Parts:
- added TP210, TP211: TestPoint, symbol Connector:TestPoint
Connections:
- net SPI_MOSI: now also TP403.1, U401.5 (DI_(IO0_))
- net SPI_SCLK: now also TP401.1, U401.1 (~{CS}), U902.5 (1A2), U903.4 (1A1)
- net at R207.2, U201.16 (SPI-ChipSelect(GPIO18)): no longer TP401.1, U401.1 (~{CS})
- net at TP404.1, U401.2 (DO_(IO1_)): no longer U201.19 (SPI_dataIn(GPIO21))
- net GNSS_UART_TX: now reaches J201.4 (Pin_4), R205.2
- net LINTXD: no longer names the net of U201.5 (LIN-transmit(GPIO5))
- net LINTXD: now also TP210.1
- net LIN_RXD: no longer names the net of U201.4 (LIN-receive(GPIO4))
- net LIN_RXD: now also TP211.1
- new net SPI_MISO: U201.19 (SPI_dataIn(GPIO21))
Other:
- note removed: "SPI_MISO"
- moved on the sheet: TP403
