File: mcu_peripherals.kicad_sch (KiCad schematic)
At the start: 77 parts, among them J201 Conn_01x05, J601 USB_C_Receptacle_USB2.0_16P, J901 Micro_SD_Card_Det_Hirose_DM3AT, SW201 BOOT, SW202 RESET, T201 TP 201, U202 TCA9535PWR, U203 TPS3840DL42DBVR, U401 W25N01GVZEIG, U601 USBLC6-2SC6, U602 USBLC6-2SC6, U702 ATECC608B-SSHDA, U801 ASM330LHHTR, U802 TMP1075DGKR, U901 TPS22918TDBVTQ1, U902 SN74AXC4T245QPWRQ1, U903 SN74AXC4T245QPWRQ1

Commit message: hierarchy
Parts:
- renumbered C214 to C44, C601 to C48, C702 to C49, C211 to C50, C212 to C51, C207 to C52, C203 to C53, C213 to C54, C201 to C55, C202 to C56, C402 to C57, C210 to C58, C401 to C59, C209 to C60, C205 to C61, C204 to C62, C206 to C63, C904 to C64, C208 to C65, C907 to C66, C908 to C67, C902 to C68, C901 to C69, D201 to D4, F106 to F2, J601 to J2, J201 to J3, J901 to J4, R801 to R1, R215 to R12, R602 to R2, R204 to R20, R203 to R22, R202 to R24, R201 to R25, R213 to R30, R207 to R34, R12 to R38, R209 to R41, R205 to R47, R206 to R48, R210 to R49, R601 to R5, R211 to R50, R401 to R51, R212 to R52, R402 to R53, R903 to R54, R904 to R55, R905 to R56, R901 to R57, R214 to R58, SW202 to SW1, SW201 to SW2, T201 to T1, TP402 to TP12, TP401 to TP13, TP403 to TP14, TP404 to TP15, TP901 to TP16, TP202 to TP17, TP601 to TP2, TP211 to TP7, TP210 to TP8, U601 to U12, U802 to U13, U203 to U14, U702 to U15, U602 to U16, U801 to U17, U202 to U18, U201 to U19, U401 to U20, U903 to U21, U902 to U22, U901 to U23

Commit message: Renaming
Parts:
- renumbered R38 to R209, T1 to TP201
Connections:
- net I2C_SDA: now reaches R24.1, U13.1 (SDA), U15.5 (SDA), U17.14 (SDA), U18.1 (~{INT}), U19.6 (I2C-data(GPIO6))
- net I2C_SCL: now reaches R22.1, U13.2 (SCL), U15.6 (SCL), U17.13 (SCL), U18.22 (SCL), U19.7 (I2C-clock(GPIO7))
Other:
- note removed: "I2C_SCL"
- note removed: "I2C_SDA"
Changed lines of the file:
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@@
 		)
 	)
-	(text "I2C_SCL"
-		(exclude_from_sim no)
-		(at 229.87 118.618 0)
-		(effects
-			(font
-				(size 1.27 1.27)
-			)
-		)
-	)
 	(text "BOOT\n"
 		(exclude_from_sim no)
@@
 		)
 	)
-	(text "I2C_SDA"
-		(exclude_from_sim no)
-		(at 229.87 112.268 0)
-		(effects
-			(font
-				(size 1.27 1.27)
-			)
-		)
-	)
 	(text "TEMP SENSOR"
 		(exclude_from_sim no)
@@
 		)
 	)
+	(label "I2C_SDA"
+		(at 224.79 113.03 0)
+		(effects
+			(font
+				(size 1.27 1.27)
+			)
+			(justify left bottom)
+		)
+	)
 	(label "CAN1_TXD"
 		(at 394.97 154.94 0)
@@
 		)
 	)
+	(label "I2C_SCL"
+		(at 224.79 119.38 0)
+		(effects
+			(font
+				(size 1.27 1.27)
+			)
+			(justify left bottom)
+		)
+	)
 	(label "USB_DN"
 		(at 394.97 147.32 0)
@@
 		(in_pos_files yes)
 		(dnp no)
-		(property "Reference" "R38"
-			(at 342.9 149.606 90)
+		(property "Reference" "R209"
+			(at 341.63 149.606 90)
 			(show_name no)
 			(do_not_autoplace no)
@@
 		)
 		(property "Value" "22"
-			(at 342.9 152.146 90)
+			(at 342.9 151.638 90)
 			(show_name no)
 			(do_not_autoplace no)
@@
 			(project "Tracker"
 				(path "/586d1ea1-b017-4713-987c-545d658f6cc8/378094db-8f3e-4510-9f4d-07bbb8577682"
-					(reference "R38")
+					(reference "R209")
 					(unit 1)
 				)
@@
 		(dnp no)
 		(fields_autoplaced yes)
-		(property "Reference" "T1"
+		(property "Reference" "TP201"
 			(at 322.58 51.3079 0)
 			(show_name no)
@@
 			(project "Tracker"
 				(path "/586d1ea1-b017-4713-987c-545d658f6cc8/378094db-8f3e-4510-9f4d-07bbb8577682"
-					(reference "T1")
+					(reference "TP201")
 					(unit 1)
 				)

Commit message: Bug fix
Connections:
- net I2C_SDA: now also U18.23 (SDA); no longer U18.1 (~{INT})
- net at R20.1, U19.27 (Expander-interrupt(GPI02)): now also U18.1 (~{INT}); no longer U18.23 (SDA)
Other:
- moved on the sheet: TP7, TP8
Changed lines of the file:
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@@
 	(wire
 		(pts
-			(xy 180.34 102.87) (xy 233.68 102.87)
+			(xy 227.33 102.87) (xy 233.68 102.87)
 		)
 		(stroke
@@
 	(wire
 		(pts
-			(xy 168.91 100.33) (xy 233.68 100.33)
+			(xy 224.79 100.33) (xy 233.68 100.33)
 		)
 		(stroke
@@
 		(in_pos_files yes)
 		(dnp no)
-		(fields_autoplaced yes)
 		(property "Reference" "#PWR018"
 			(at 204.47 279.4 0)
@@
 		)
 		(property "Value" "GND"
-			(at 204.47 278.13 0)
+			(at 206.248 276.86 0)
 			(show_name no)
 			(do_not_autoplace no)
@@
 	(symbol
 		(lib_id "Connector:TestPoint")
-		(at 180.34 102.87 180)
+		(at 227.33 102.87 180)
 		(unit 1)
 		(body_style 1)
@@
 		(dnp no)
 		(property "Reference" "TP8"
-			(at 178.308 108.458 0)
+			(at 229.362 106.426 0)
 			(show_name no)
 			(do_not_autoplace no)
@@
 		)
 		(property "Value" "TestPoint"
-			(at 182.88 107.4419 0)
+			(at 229.87 107.4419 0)
 			(hide yes)
 			(show_name no)
@@
 		)
 		(property "Footprint" ""
-			(at 175.26 102.87 0)
+			(at 222.25 102.87 0)
 			(hide yes)
 			(show_name no)
@@
 		)
 		(property "Datasheet" ""
-			(at 175.26 102.87 0)
+			(at 222.25 102.87 0)
 			(hide yes)
 			(show_name no)
@@
 		)
 		(property "Description" "test point"
-			(at 180.34 102.87 0)
+			(at 227.33 102.87 0)
 			(hide yes)
 			(show_name no)
@@
 	(symbol
 		(lib_id "Connector:TestPoint")
-		(at 168.91 100.33 180)
+		(at 224.79 100.33 180)
 		(unit 1)
 		(body_style 1)
@@
 		(dnp no)
 		(property "Reference" "TP7"
-			(at 166.624 105.918 0)
+			(at 219.71 104.14 0)
 			(show_name no)
 			(do_not_autoplace no)
@@
 		)
 		(property "Value" "TestPoint"
-			(at 171.45 104.9019 0)
+			(at 227.33 104.9019 0)
 			(hide yes)
 			(show_name no)
@@
 		)
 		(property "Footprint" ""
-			(at 163.83 100.33 0)
+			(at 219.71 100.33 0)
 			(hide yes)
 			(show_name no)
@@
 		)
 		(property "Datasheet" ""
-			(at 163.83 100.33 0)
+			(at 219.71 100.33 0)
 			(hide yes)
 			(show_name no)
@@
 		)
 		(property "Description" "test point"
-			(at 168.91 100.33 0)
+			(at 224.79 100.33 0)
 			(hide yes)
 			(show_name no)
@@
 		(in_pos_files yes)
 		(dnp no)
-		(fields_autoplaced yes)
 		(property "Reference" "#PWR019"
 			(at 180.34 271.78 0)
@@
 		)
 		(property "Value" "GND"
-			(at 180.34 270.51 0)
+			(at 180.34 269.748 0)
 			(show_name no)
 			(do_not_autoplace no)

Commit message: bug
Parts:
- R202: renamed from R20; value 2.2k -> 10k
- R203: renamed from R24; value 10k -> 2.2k
- renumbered R22 to R204
Connections:
- net SPI_MISO: now also TP15.1, U20.2 (DO_(IO1_))
Other:
- moved on the sheet: TP15
Changed lines of the file:
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@@
 	(text "SPI_CS0_N"
 		(exclude_from_sim no)
-		(at 306.832 117.094 0)
+		(at 314.198 117.094 0)
 		(effects
 			(font
@@
 	)
 	(junction
+		(at 300.99 110.49)
+		(diameter 0)
+		(color 0 0 0 0)
+	)
+	(junction
 		(at 401.32 223.52)
 		(diameter 0)
@@
 	)
 	(junction
-		(at 396.24 368.3)
-		(diameter 0)
-		(color 0 0 0 0)
-	)
-	(junction
 		(at 364.49 223.52)
 		(diameter 0)
@@
 	)
 	(junction
+		(at 386.08 368.3)
+		(diameter 0)
+		(color 0 0 0 0)
+	)
+	(junction
 		(at 172.72 361.95)
 		(diameter 0)
@@
 	(wire
 		(pts
-			(xy 327.66 355.6) (xy 330.2 355.6)
+			(xy 123.19 147.32) (xy 156.21 147.32)
 		)
 		(stroke
@@
 	(wire
 		(pts
-			(xy 123.19 147.32) (xy 156.21 147.32)
+			(xy 461.01 209.55) (xy 461.01 220.98)
 		)
 		(stroke
@@
 	(wire
 		(pts
-			(xy 461.01 209.55) (xy 461.01 220.98)
+			(xy 401.32 223.52) (xy 406.4 223.52)
 		)
 		(stroke
@@
 	(wire
 		(pts
-			(xy 401.32 223.52) (xy 406.4 223.52)
+			(xy 222.25 229.87) (xy 248.92 229.87)
 		)
 		(stroke
@@
 	(wire
 		(pts
-			(xy 222.25 229.87) (xy 248.92 229.87)
+			(xy 364.49 220.98) (xy 364.49 223.52)
 		)
 		(stroke
@@
 	(wire
 		(pts
-			(xy 364.49 220.98) (xy 364.49 223.52)
+			(xy 336.55 128.27) (xy 336.55 147.32)
 		)
 		(stroke
@@
 	(wire
 		(pts
-			(xy 336.55 128.27) (xy 336.55 147.32)
+			(xy 300.99 355.6) (xy 330.2 355.6)
 		)
 		(stroke
@@
 	(wire
 		(pts
+			(xy 386.08 383.54) (xy 303.53 383.54)
+		)
+		(stroke
+			(width 0)
+			(type default)
+		)
+	)
+	(wire
+		(pts
 			(xy 60.96 271.78) (xy 62.23 271.78)
 		)
@@
 	(wire
 		(pts
+			(xy 300.99 110.49) (xy 303.53 110.49)
+		)
+		(stroke
+			(width 0)
+			(type default)
+		)
+	)
+	(wire
+		(pts
 			(xy 359.41 330.2) (xy 344.17 330.2)
 		)
@@
 	(wire
 		(pts
-			(xy 382.27 368.3) (xy 396.24 368.3)
+			(xy 382.27 368.3) (xy 386.08 368.3)
 		)
 		(stroke
@@
 	(wire
 		(pts
-			(xy 400.05 384.81) (xy 400.05 368.3)
-		)
-		(stroke
-			(width 0)
-			(type default)
-		)
-	)
-	(wire
-		(pts
 			(xy 156.21 205.74) (xy 156.21 229.87)
 		)
@@
 	(wire
 		(pts
-			(xy 297.18 384.81) (xy 400.05 384.81)
-		)
-		(stroke
-			(width 0)
-			(type default)
-		)
-	)
-	(wire
-		(pts
 			(xy 161.29 335.28) (xy 173.99 335.28)
 		)
@@
 	(wire
 		(pts
+			(xy 303.53 113.03) (xy 303.53 383.54)
+		)
+		(stroke
+			(width 0)
+			(type default)
+		)
+	)
+	(wire
+		(pts
 			(xy 377.19 275.59) (xy 378.46 275.59)
 		)
@@
 	(wire
 		(pts
-			(xy 293.37 110.49) (xy 303.53 110.49)
+			(xy 293.37 110.49) (xy 300.99 110.49)
 		)
 		(stroke
@@
 	(wire
 		(pts
+			(xy 386.08 368.3) (xy 386.08 383.54)
+		)
+		(stroke
+			(width 0)
+			(type default)
+		)
+	)
+	(wire
+		(pts
 			(xy 364.49 218.44) (xy 367.03 218.44)
 		)
@@
 	(wire
 		(pts
-			(xy 396.24 368.3) (xy 400.05 368.3)
-		)
-		(stroke
-			(width 0)
-			(type default)
-		)
-	)
-	(wire
-		(pts
 			(xy 336.55 147.32) (xy 340.36 147.32)
 		)
@@
 	(wire
 		(pts
+			(xy 300.99 110.49) (xy 300.99 355.6)
+		)
+		(stroke
+			(width 0)
+			(type default)
+		)
+	)
+	(wire
+		(pts
 			(xy 325.12 182.88) (xy 419.1 182.88)
 		)
@@
 		)
 	)
-	(label "I2C_SDA"
-		(at 224.79 113.03 0)
-		(effects
-			(font
-				(size 1.27 1.27)
-			)
-			(justify left bottom)
-		)
-	)
 	(label "CAN1_TXD"
 		(at 394.97 154.94 0)
@@
 		)
 	)
-	(label "I2C_SCL"
-		(at 224.79 119.38 0)
-		(effects
-			(font
-				(size 1.27 1.27)
-			)
-			(justify left bottom)
-		)
-	)
 	(label "USB_DN"
 		(at 394.97 147.32 0)
@@
 		)
 	)
+	(global_label "I2C_SDA"
+		(shape bidirectional)
+		(at 222.25 113.03 0)
+		(fields_autoplaced yes)
+		(effects
+			(font
+				(size 1.27 1.27)
+			)
+			(justify left)
+		)
+		(property "Intersheetrefs" "${INTERSHEET_REFS}"
+			(at 233.9665 113.03 0)
+			(hide yes)
+			(show_name no)
+			(do_not_autoplace no)
+			(effects
+				(font
+					(size 1.27 1.27)
+				)
+				(justify left)
+			)
+		)
+	)
 	(global_label "VSUP_SENSE"
 		(shape input)
@@
 		)
 	)
+	(global_label "I2C_SCL"
+		(shape bidirectional)
+		(at 232.41 119.38 180)
+		(fields_autoplaced yes)
+		(effects
+			(font
+				(size 1.27 1.27)
+			)
+			(justify right)
+		)
+		(property "Intersheetrefs" "${INTERSHEET_REFS}"
+			(at 220.754 119.38 0)
+			(hide yes)
+			(show_name no)
+			(do_not_autoplace no)
+			(effects
+				(font
+					(size 1.27 1.27)
+				)
+				(justify right)
+			)
+		)
+	)
 	(global_label "VIN_SENSE"
 		(shape input)
@@
 		(dnp no)
 		(fields_autoplaced yes)
-		(property "Reference" "R20"
+		(property "Reference" "R202"
 			(at 199.39 132.0799 0)
 			(show_name no)
@@
 			)
 		)
-		(property "Value" "2.2k"
+		(property "Value" "10k"
 			(at 199.39 134.6199 0)
 			(show_name no)
@@
 			(project "Tracker"
 				(path "/586d1ea1-b017-4713-987c-545d658f6cc8/378094db-8f3e-4510-9f4d-07bbb8577682"
-					(reference "R20")
+					(reference "R202")
 					(unit 1)
 				)
@@
 		(dnp no)
 		(fields_autoplaced yes)
-		(property "Reference" "R24"
+		(property "Reference" "R203"
 			(at 222.25 132.0799 0)
 			(show_name no)
@@
 			)
 		)
-		(property "Value" "10k"
+		(property "Value" "2.2k"
 			(at 222.25 134.6199 0)
 			(show_name no)
@@
 			(project "Tracker"
 				(path "/586d1ea1-b017-4713-987c-545d658f6cc8/378094db-8f3e-4510-9f4d-07bbb8577682"
-					(reference "R24")
+					(reference "R203")
 					(unit 1)
 				)
@@
 	(symbol
 		(lib_id "Connector:TestPoint")
-		(at 396.24 368.3 0)
+		(at 386.08 368.3 0)
 		(unit 1)
 		(body_style 1)
@@
 		(fields_autoplaced yes)
 		(property "Reference" "TP15"
-			(at 398.78 363.7279 0)
+			(at 388.62 363.7279 0)
 			(show_name no)
 			(do_not_autoplace no)
@@
 		)
 		(property "Value" "TP 404"
-			(at 398.78 366.2679 0)
+			(at 388.62 366.2679 0)
 			(show_name no)
 			(do_not_autoplace no)
@@
 		)
 		(property "Footprint" ""
-			(at 401.32 368.3 0)
+			(at 391.16 368.3 0)
 			(hide yes)
 			(show_name no)
@@
 		)
 		(property "Datasheet" ""
-			(at 401.32 368.3 0)
+			(at 391.16 368.3 0)
 			(hide yes)
 			(show_name no)
@@
 		)
 		(property "Description" "test point"
-			(at 396.24 368.3 0)
+			(at 386.08 368.3 0)
 			(hide yes)
 			(show_name no)
@@
 		(dnp no)
 		(fields_autoplaced yes)
-		(property "Reference" "R22"
+		(property "Reference" "R204"
 			(at 210.82 132.0799 0)
 			(show_name no)
@@
 			(project "Tracker"
 				(path "/586d1ea1-b017-4713-987c-545d658f6cc8/378094db-8f3e-4510-9f4d-07bbb8577682"
-					(reference "R22")
+					(reference "R204")
 					(unit 1)
 				)
@@
 		(dnp no)
 		(property "Reference" "R47"
-			(at 354.33 81.2799 90)
+			(at 350.52 86.106 90)
 			(show_name no)
 			(do_not_autoplace no)
@@
 		)
 		(property "Value" "499"
-			(at 354.33 83.8199 90)
+			(at 355.092 87.63 90)
 			(show_name no)
 			(do_not_autoplace no)

Commit message: bug fix
Parts:
- removed TP8: TestPoint, symbol Connector:TestPoint
- added R20: 100k, symbol Device:R
- added R22, R24, R38: 10k, symbol Device:R
- added TP204, TP205, TP210: TestPoint, symbol Connector:TestPoint
- renumbered TP7 to TP211, TP14 to TP403, U22 to U902, U21 to U903
Connections:
- net 3V3_AUX: now also U23.1 (VIN); no longer U23.6 (VOUT)
- net BUCK_PG: now also R20.2; no longer U18.5 (P01)
- net CHG_INT_N: now also R24.2; no longer U18.7 (P03)
- net GND: now also U23.2 (GND); no longer U23.5 (QOD)
- net I2C_SCL: now also TP204.1
- net I2C_SDA: now also TP205.1
- net MUX_ST: now also R22.2; no longer U18.6 (P02)
- net PM_ALERT_N: now also R38.2; no longer U18.8 (P04)
- net SPI_MOSI: now also U902.5 (1A2)
- net SPI_SCLK: now also TP12.1, U20.6 (CLK), U902.4 (1A1); no longer TP13.1, U20.1 (~{CS}), U902.5 (1A2)
- net at C64.2, C66.1, C67.1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: now also U23.5 (QOD), U23.6 (VOUT); no longer U23.1 (VIN), U23.2 (GND)
- net at R41.1: now also U19.14 (USB_D+(GPIO13)); no longer U19.13 (USB_D-(GPIO12))
- net SD_CS_N: now reaches U902.6 (2A1), U903.15 (1~{OE})
- net SD_CS_N: now also U19.5 (LIN-transmit(GPIO5)), TP210.1
- net at R209.1: now also U19.13 (USB_D-(GPIO12)); no longer U19.14 (USB_D+(GPIO13))
- new net: R22.1, U18.6 (P02)
- new net: R38.1, U18.8 (P04)
- new net: R24.1, U18.7 (P03)
- new net: R20.1, U18.5 (P01)
- new net SPI_CSO_N: TP13.1, U20.1 (~{CS})
Other:
- moved on the sheet: TP211, U23

Commit message: Fix SD card net and designator cleanup
This commit renumbers a few schematic components and fixes the SD-card interface wiring in the MCU and cellular sheets. It updates the DAT1/DAT2 pin directions and net labels, adds the missing power/junction connections for the SD rail, and aligns pull-up resistors and capacitor values with the revised SD_VDD routing. Related KiCad designator and power-symbol cleanup was also applied to keep the schematic consistent.
Parts:
- added R904, R905: 47K, symbol Device:R
- C57: value 1nF -> 1uF
- C59: value 100uF -> 10uF
- renumbered R2 to R601, R5 to R602, R1 to R801, U13 to U802
Connections:
- net 3V3_AON: now also U902.2 (1DIR), U902.3 (2DIR); no longer C65.1, U902.16 (VCCB)
- net GND: now also D1.2 (A2); no longer D1.1 (A1), U902.2 (1DIR), U902.3 (2DIR)
- net SD_VDD: now also C64.2, C65.1, C66.1, C67.1, J4.4 (VDD), TP16.1, U23.5 (QOD), U23.6 (VOUT), U902.16 (VCCB), U903.16 (VCCB), R904.2, R905.2
- net VBUS_USB: now also D1.1 (A1); no longer D1.2 (A2)
- net SD_DAT2: now reaches J4.1 (DAT2)
- net SD_DAT2: now also R904.1
- net SD_DAT1: now reaches J4.8 (DAT1)
- net SD_DAT1: now also R905.1
- net SPI_CSO_N renamed SPI_CS0_N
Other:
- moved on the sheet: C66, C67, R55, R56, TP16
