File: mcu_peripherals.kicad_sch (KiCad schematic)
At the start: 87 parts, among them J2 USB_C_Receptacle_USB2.0_16P, J3 Conn_01x05, J4 Micro_SD_Card_Det_Hirose_DM3AT, SW1 RESET, SW2 BOOT, U12 USBLC6-2SC6, U14 TPS3840DL42DBVR, U15 ATECC608B-SSHDA, U16 USBLC6-2SC6, U17 ASM330LHHTR, U18 TCA9535PWR, U20 W25N01GVZEIG, U23 TPS22918TDBVTQ1, U802 TMP1075DGKR, U902 SN74AXC4T245QPWRQ1, U903 SN74AXC4T245QPWRQ1

Commit message: bug fix
Parts:
- removed U14: TPS3840DL42DBVR, SamacSys_Parts:SOT95P280X145-6N, symbol TPS3840DL42DBVR:TPS3840DL42DBVR
- added TP14: TestPoint, SOT95P280X145-5N, symbol Connector:TestPoint
- added U14: TPS3840DL30DBVR, SOT95P280X145-5N, symbol SamacSys_Parts:TPS3840DL30DBVR
Connections:
- net 3V3_AON: now also U14.2 (VDD), U14.4 (~{MR_}/_NC)
- net GND: now also U14.3 (GND)
- net at C53.1, J3.2 (Pin_2), R12.2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: now also TP14.1
- net TEMP_ALERT_N: now reaches R801.1, U802.3 (ALERT)
- net at R12.1: now also U14.1 (~{RESET})
Other:
- note removed: "TEMP_ALERT_N"

Commit message: Footprint
Parts:
- C48: footprint (none) -> Capacitor_SMD:C_0805_2012Metric
- C49: footprint (none) -> Capacitor_SMD:C_0402_1005Metric
- J3: footprint (none) -> Connector_PinSocket_2.54mm:PinSocket_1x05_P2.54mm_Vertical
- J4, U902, U903: footprint SOP65P640X120-16N -> SamacSys_Parts:SOP65P640X120-16N
- R12: value 1K -> DNP; footprint (none) -> Resistor_SMD:R_0603_1608Metric
- R20, R202, R203, R204, R205, R209, R22, R24, R25, R30, R34, R41, R48, R49, R50, R52, R58: footprint (none) -> Resistor_SMD:R_0603_1608Metric
- R201, R51, R53, R54, R55, R56, R57, R801, R904, R905, R906: footprint (none) -> Resistor_SMD:R_0402_1005Metric
- R38: footprint (none) -> Rotary_Encoder:RotaryEncoder_Bourns_Horizontal_PEL12D-2x18F-Sxxxx
- R601, R602: footprint Package_DIP:DIP-8_W7.62mm -> Resistor_SMD:R_1206_3216Metric
- SW1, SW2: footprint Button_Switch_THT:SW_NKK_GW12LJP -> Button_Switch_SMD:SW_SPST_TL3342
- TP12, TP13, TP15, TP16, TP2, TP201, TP204, TP205, TP210, TP211, TP403: footprint (none) -> TestPoint:TestPoint_Pad_D1.5mm
- TP14: footprint SOT95P280X145-5N -> TestPoint:TestPoint_Pad_D1.5mm
- TP17: footprint Relay_THT:Relay_DPDT_Schrack-RT2-FormC_RM5mm -> TestPoint:TestPoint_Pad_D1.5mm
- U14: footprint SOT95P280X145-5N -> SamacSys_Parts:SOT95P280X145-5N
- U20: footprint SON127P800X600X80-9N-D -> SamacSys_Parts:SON127P800X600X80-9N-D
- U23: footprint SOT95P280X145-6N -> SamacSys_Parts:SOT95P280X145-6N
- U802: footprint DGK0008A_N -> Package_SO:VSSOP-8_3x3mm_P0.65mm
Other:
- moved on the sheet: C62, R48

Commit message: Footprint
Parts:
- C44, C53: footprint RF_Module:ESP32-C6-MINI-1 -> Capacitor_SMD:C_0603_1608Metric
- C50, C51, C52, C54, C56, C57, C58, C60, C61, C62, C63, C64, C65, C67, C68, C69: footprint RF_Module:ESP32-C6-MINI-1 -> Capacitor_SMD:C_0402_1005Metric
- C55, C66: footprint RF_Module:ESP32-C6-MINI-1 -> Capacitor_SMD:C_0805_2012Metric
- C59: value 10uF -> 10nF; footprint RF_Module:ESP32-C6-MINI-1 -> Capacitor_SMD:C_0402_1005Metric
- D4: footprint LED_SMD:LED_Cree-XHP50_3V_HighDensity -> LED_SMD:LED_0603_1608Metric
- F2: footprint Package_LCC:PLCC-84_29.3x29.3mm_P1.27mm -> Fuse:Fuse_1206_3216Metric
- J2: footprint Package_DFN_QFN:WDFN-10-1EP_3x3mm_P0.5mm_EP1.8x2.5mm -> Connector_USB:USB_C_Receptacle_GCT_USB4105-xx-A_16P_TopMnt_Horizontal
- J4: footprint SamacSys_Parts:SOP65P640X120-16N -> Connector_Card:microSD_HC_Hirose_DM3AT-SF-PEJM5
- R38: footprint Rotary_Encoder:RotaryEncoder_Bourns_Horizontal_PEL12D-2x18F-Sxxxx -> Resistor_SMD:R_0603_1608Metric
Other:
- moved on the sheet: TP403
Changed lines of the file:
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@@
 	)
 	(junction
-		(at 330.2 355.6)
+		(at 323.85 355.6)
 		(diameter 0)
 		(color 0 0 0 0)
@@
 	(wire
 		(pts
-			(xy 313.69 355.6) (xy 330.2 355.6)
+			(xy 313.69 355.6) (xy 336.55 355.6)
 		)
 		(stroke
@@
 	(wire
 		(pts
-			(xy 330.2 355.6) (xy 336.55 355.6)
-		)
-		(stroke
-			(width 0)
-			(type default)
-		)
-	)
-	(wire
-		(pts
 			(xy 293.37 92.71) (xy 300.99 92.71)
 		)
@@
 			)
 		)
-		(property "Footprint" "SamacSys_Parts:SOP65P640X120-16N"
+		(property "Footprint" "Connector_Card:microSD_HC_Hirose_DM3AT-SF-PEJM5"
 			(at 537.21 240.03 0)
 			(hide yes)
@@
 			)
 		)
-		(property "Footprint" "RF_Module:ESP32-C6-MINI-1"
+		(property "Footprint" "Capacitor_SMD:C_0402_1005Metric"
 			(at 310.8452 63.5 0)
 			(hide yes)
@@
 			)
 		)
-		(property "Footprint" "RF_Module:ESP32-C6-MINI-1"
+		(property "Footprint" "Capacitor_SMD:C_0402_1005Metric"
 			(at 381.9652 105.41 0)
 			(hide yes)
@@
 			)
 		)
-		(property "Footprint" "Rotary_Encoder:RotaryEncoder_Bourns_Horizontal_PEL12D-2x18F-Sxxxx"
+		(property "Footprint" "Resistor_SMD:R_0603_1608Metric"
 			(at 246.888 210.82 90)
 			(hide yes)
@@
 			)
 		)
-		(property "Footprint" "RF_Module:ESP32-C6-MINI-1"
+		(property "Footprint" "Capacitor_SMD:C_0402_1005Metric"
 			(at 181.3052 316.23 0)
 			(hide yes)
@@
 			)
 		)
-		(property "Footprint" "RF_Module:ESP32-C6-MINI-1"
+		(property "Footprint" "Capacitor_SMD:C_0402_1005Metric"
 			(at 389.5852 283.21 0)
 			(hide yes)
@@
 			)
 		)
-		(property "Footprint" "Package_DFN_QFN:WDFN-10-1EP_3x3mm_P0.5mm_EP1.8x2.5mm"
+		(property "Footprint" "Connector_USB:USB_C_Receptacle_GCT_USB4105-xx-A_16P_TopMnt_Horizontal"
 			(at 49.53 274.32 0)
 			(hide yes)
@@
 			)
 		)
-		(property "Footprint" "Package_LCC:PLCC-84_29.3x29.3mm_P1.27mm"
+		(property "Footprint" "Fuse:Fuse_1206_3216Metric"
 			(at 68.58 251.968 90)
 			(hide yes)
@@
 			)
 		)
-		(property "Footprint" "RF_Module:ESP32-C6-MINI-1"
+		(property "Footprint" "Capacitor_SMD:C_0402_1005Metric"
 			(at 345.7448 215.9 0)
 			(hide yes)
@@
 			)
 		)
-		(property "Footprint" "RF_Module:ESP32-C6-MINI-1"
+		(property "Footprint" "Capacitor_SMD:C_0402_1005Metric"
 			(at 385.7752 135.89 0)
 			(hide yes)
@@
 			)
 		)
-		(property "Footprint" "RF_Module:ESP32-C6-MINI-1"
+		(property "Footprint" "Capacitor_SMD:C_0402_1005Metric"
 			(at 360.9848 139.7 0)
 			(hide yes)
@@
 			)
 		)
-		(property "Footprint" "RF_Module:ESP32-C6-MINI-1"
+		(property "Footprint" "Capacitor_SMD:C_0402_1005Metric"
 			(at 416.2552 226.06 0)
 			(hide yes)
@@
 			)
 		)
-		(property "Footprint" "RF_Module:ESP32-C6-MINI-1"
+		(property "Footprint" "Capacitor_SMD:C_0402_1005Metric"
 			(at 329.2348 330.2 0)
 			(hide yes)
@@
 			)
 		)
-		(property "Footprint" "RF_Module:ESP32-C6-MINI-1"
+		(property "Footprint" "Capacitor_SMD:C_0805_2012Metric"
 			(at 436.5752 237.49 0)
 			(hide yes)
@@
 			)
 		)
-		(property "Footprint" "RF_Module:ESP32-C6-MINI-1"
+		(property "Footprint" "Capacitor_SMD:C_0402_1005Metric"
 			(at 514.0452 213.36 0)
 			(hide yes)
@@
 			)
 		)
-		(property "Footprint" "RF_Module:ESP32-C6-MINI-1"
+		(property "Footprint" "Capacitor_SMD:C_0402_1005Metric"
 			(at 450.5452 237.49 0)
 			(hide yes)
@@
 			)
 		)
-		(property "Footprint" "RF_Module:ESP32-C6-MINI-1"
+		(property "Footprint" "Capacitor_SMD:C_0603_1608Metric"
 			(at 199.6948 80.01 0)
 			(hide yes)
@@
 			)
 		)
-		(property "Footprint" "RF_Module:ESP32-C6-MINI-1"
+		(property "Footprint" "Capacitor_SMD:C_0402_1005Metric"
 			(at 186.3852 217.17 0)
 			(hide yes)
@@
 			)
 		)
-		(property "Footprint" "RF_Module:ESP32-C6-MINI-1"
+		(property "Footprint" "Capacitor_SMD:C_0402_1005Metric"
 			(at 494.9952 218.44 0)
 			(hide yes)
@@
 			)
 		)
-		(property "Value" "10uF"
+		(property "Value" "10nF"
 			(at 341.122 331.978 0)
 			(show_name no)
@@
 			)
 		)
-		(property "Footprint" "RF_Module:ESP32-C6-MINI-1"
+		(property "Footprint" "Capacitor_SMD:C_0402_1005Metric"
 			(at 343.2048 330.2 0)
 			(hide yes)
@@
 			)
 		)
-		(property "Footprint" "RF_Module:ESP32-C6-MINI-1"
+		(property "Footprint" "Capacitor_SMD:C_0402_1005Metric"
 			(at 172.4152 316.23 0)
 			(hide yes)
@@
 			)
 		)
-		(property "Footprint" "RF_Module:ESP32-C6-MINI-1"
+		(property "Footprint" "Capacitor_SMD:C_0402_1005Metric"
 			(at 327.9648 281.94 0)
 			(hide yes)
@@
 			)
 		)
-		(property "Footprint" "LED_SMD:LED_Cree-XHP50_3V_HighDensity"
+		(property "Footprint" "LED_SMD:LED_0603_1608Metric"
 			(at 453.39 132.08 0)
 			(hide yes)
@@
 	(symbol
 		(lib_id "Connector:TestPoint")
-		(at 330.2 355.6 0)
+		(at 323.85 355.6 0)
 		(unit 1)
 		(body_style 1)
@@
 		(dnp no)
 		(property "Reference" "TP403"
-			(at 331.47 350.52 0)
+			(at 325.12 350.52 0)
 			(show_name no)
 			(do_not_autoplace no)
@@
 		)
 		(property "Value" "TP 403"
-			(at 331.47 353.06 0)
+			(at 325.12 353.06 0)
 			(show_name no)
 			(do_not_autoplace no)
@@
 		)
 		(property "Footprint" "TestPoint:TestPoint_Pad_D1.5mm"
-			(at 335.28 355.6 0)
+			(at 328.93 355.6 0)
 			(hide yes)
 			(show_name no)
@@
 		)
 		(property "Datasheet" ""
-			(at 335.28 355.6 0)
+			(at 328.93 355.6 0)
 			(hide yes)
 			(show_name no)
@@
 		)
 		(property "Description" "test point"
-			(at 330.2 355.6 0)
+			(at 323.85 355.6 0)
 			(hide yes)
 			(show_name no)
@@
 			)
 		)
-		(property "Footprint" "RF_Module:ESP32-C6-MINI-1"
+		(property "Footprint" "Capacitor_SMD:C_0402_1005Metric"
 			(at 202.8952 316.23 0)
 			(hide yes)
@@
 			)
 		)
-		(property "Footprint" "RF_Module:ESP32-C6-MINI-1"
+		(property "Footprint" "Capacitor_SMD:C_0603_1608Metric"
 			(at 87.9348 140.97 0)
 			(hide yes)
@@
 			)
 		)
-		(property "Footprint" "RF_Module:ESP32-C6-MINI-1"
+		(property "Footprint" "Capacitor_SMD:C_0805_2012Metric"
 			(at 296.8752 63.5 0)
 			(hide yes)

Commit message: Update fix
Parts:
- U12, U16: symbol Power_Protection:USBLC6-2SC6 -> Project_Parts:USBLC6-2SC6
- U18: symbol Interface_Expansion:TCA9535PWR -> Project_Parts:TCA9535PWR
- U802: symbol 2026-10-02_18-26-52:TMP1075DGKR -> Project_Parts:TMP1075DGKR
Changed lines of the file:
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@@
 	)
 	(symbol
-		(lib_id "power:GND")
+		(lib_id "gnd_NoFootPrint:GND")
 		(at 328.93 289.56 0)
 		(unit 1)
@@
 	)
 	(symbol
-		(lib_id "power:GND")
+		(lib_id "gnd_NoFootPrint:GND")
 		(at 204.47 273.05 0)
 		(unit 1)
@@
 	)
 	(symbol
-		(lib_id "power:GND")
+		(lib_id "gnd_NoFootPrint:GND")
 		(at 96.52 303.53 0)
 		(unit 1)
@@
 	)
 	(symbol
-		(lib_id "power:GND")
+		(lib_id "gnd_NoFootPrint:GND")
 		(at 200.66 80.01 180)
 		(unit 1)
@@
 	)
 	(symbol
-		(lib_id "power:GND")
+		(lib_id "gnd_NoFootPrint:GND")
 		(at 342.9 275.59 0)
 		(unit 1)
@@
 	)
 	(symbol
-		(lib_id "power:GND")
+		(lib_id "gnd_NoFootPrint:GND")
 		(at 361.95 139.7 180)
 		(unit 1)
@@
 	)
 	(symbol
-		(lib_id "power:GND")
+		(lib_id "gnd_NoFootPrint:GND")
 		(at 295.91 63.5 0)
 		(unit 1)
@@
 	)
 	(symbol
-		(lib_id "power:GND")
+		(lib_id "gnd_NoFootPrint:GND")
 		(at 379.73 290.83 0)
 		(unit 1)
@@
 	)
 	(symbol
-		(lib_id "power:GND")
+		(lib_id "gnd_NoFootPrint:GND")
 		(at 76.2 257.81 0)
 		(unit 1)
@@
 	)
 	(symbol
-		(lib_id "power:GND")
+		(lib_id "gnd_NoFootPrint:GND")
 		(at 388.62 290.83 0)
 		(mirror y)
@@
 	)
 	(symbol
-		(lib_id "power:GND")
+		(lib_id "gnd_NoFootPrint:GND")
 		(at 127 303.53 0)
 		(unit 1)
@@
 	)
 	(symbol
-		(lib_id "power:GND")
+		(lib_id "gnd_NoFootPrint:GND")
 		(at 180.34 316.23 0)
 		(unit 1)
@@
 	)
 	(symbol
-		(lib_id "Power_Protection:USBLC6-2SC6")
+		(lib_id "Project_Parts:USBLC6-2SC6")
 		(at 96.52 295.91 0)
 		(unit 1)
@@
 	)
 	(symbol
-		(lib_id "power:GND")
+		(lib_id "gnd_NoFootPrint:GND")
 		(at 346.71 290.83 0)
 		(unit 1)
@@
 	)
 	(symbol
-		(lib_id "power:GND")
+		(lib_id "gnd_NoFootPrint:GND")
 		(at 171.45 316.23 0)
 		(unit 1)
@@
 	)
 	(symbol
-		(lib_id "power:GND")
+		(lib_id "gnd_NoFootPrint:GND")
 		(at 415.29 226.06 0)
 		(unit 1)
@@
 	)
 	(symbol
-		(lib_id "power:GND")
+		(lib_id "gnd_NoFootPrint:GND")
 		(at 397.51 236.22 0)
 		(unit 1)
@@
 	)
 	(symbol
-		(lib_id "power:GND")
+		(lib_id "gnd_NoFootPrint:GND")
 		(at 435.61 237.49 0)
 		(unit 1)
@@
 	)
 	(symbol
-		(lib_id "power:GND")
+		(lib_id "gnd_NoFootPrint:GND")
 		(at 104.14 208.28 0)
 		(mirror y)
@@
 	)
 	(symbol
-		(lib_id "power:GND")
+		(lib_id "gnd_NoFootPrint:GND")
 		(at 449.58 237.49 0)
 		(unit 1)
@@
 	)
 	(symbol
-		(lib_id "power:GND")
+		(lib_id "gnd_NoFootPrint:GND")
 		(at 191.77 370.84 0)
 		(unit 1)
@@
 	)
 	(symbol
-		(lib_id "power:GND")
+		(lib_id "gnd_NoFootPrint:GND")
 		(at 185.42 217.17 0)
 		(unit 1)
@@
 	)
 	(symbol
-		(lib_id "power:GND")
+		(lib_id "gnd_NoFootPrint:GND")
 		(at 261.62 165.1 0)
 		(unit 1)
@@
 	)
 	(symbol
-		(lib_id "power:GND")
+		(lib_id "gnd_NoFootPrint:GND")
 		(at 356.87 378.46 0)
 		(unit 1)
@@
 	)
 	(symbol
-		(lib_id "Power_Protection:USBLC6-2SC6")
+		(lib_id "Project_Parts:USBLC6-2SC6")
 		(at 127 295.91 0)
 		(unit 1)
@@
 	)
 	(symbol
-		(lib_id "power:GND")
+		(lib_id "gnd_NoFootPrint:GND")
 		(at 124.46 160.02 0)
 		(mirror y)
@@
 	)
 	(symbol
-		(lib_id "power:GND")
+		(lib_id "gnd_NoFootPrint:GND")
 		(at 201.93 316.23 0)
 		(unit 1)
@@
 	)
 	(symbol
-		(lib_id "power:GND")
+		(lib_id "gnd_NoFootPrint:GND")
 		(at 87.63 158.75 0)
 		(mirror y)
@@
 	)
 	(symbol
-		(lib_id "power:GND")
+		(lib_id "gnd_NoFootPrint:GND")
 		(at 461.01 267.97 0)
 		(unit 1)
@@
 	)
 	(symbol
-		(lib_id "power:GND")
+		(lib_id "gnd_NoFootPrint:GND")
 		(at 452.12 111.76 0)
 		(unit 1)
@@
 	)
 	(symbol
-		(lib_id "2026-10-02_18-26-52:TMP1075DGKR")
+		(lib_id "Project_Parts:TMP1075DGKR")
 		(at 105.41 151.13 0)
 		(mirror y)
@@
 	)
 	(symbol
-		(lib_id "power:GND")
+		(lib_id "gnd_NoFootPrint:GND")
 		(at 367.03 236.22 0)
 		(unit 1)
@@
 	)
 	(symbol
-		(lib_id "power:GND")
+		(lib_id "gnd_NoFootPrint:GND")
 		(at 180.34 265.43 0)
 		(unit 1)
@@
 	)
 	(symbol
-		(lib_id "power:GND")
+		(lib_id "gnd_NoFootPrint:GND")
 		(at 45.72 297.18 0)
 		(unit 1)
@@
 	)
 	(symbol
-		(lib_id "power:GND")
+		(lib_id "gnd_NoFootPrint:GND")
 		(at 88.9 140.97 0)
 		(mirror y)
@@
 	)
 	(symbol
-		(lib_id "power:GND")
+		(lib_id "gnd_NoFootPrint:GND")
 		(at 505.46 270.51 0)
 		(unit 1)
@@
 	)
 	(symbol
-		(lib_id "power:GND")
+		(lib_id "gnd_NoFootPrint:GND")
 		(at 447.04 213.36 0)
 		(mirror y)
@@
 	)
 	(symbol
-		(lib_id "power:GND")
+		(lib_id "gnd_NoFootPrint:GND")
 		(at 38.1 297.18 0)
 		(unit 1)
@@
 	)
 	(symbol
-		(lib_id "power:GND")
+		(lib_id "gnd_NoFootPrint:GND")
 		(at 116.84 215.9 0)
 		(mirror y)
@@
 	)
 	(symbol
-		(lib_id "power:GND")
+		(lib_id "gnd_NoFootPrint:GND")
 		(at 477.52 219.71 0)
 		(unit 1)
@@
 	)
 	(symbol
-		(lib_id "power:GND")
+		(lib_id "gnd_NoFootPrint:GND")
 		(at 78.74 276.86 0)
 		(unit 1)
@@
 	)
 	(symbol
-		(lib_id "power:GND")
+		(lib_id "gnd_NoFootPrint:GND")
 		(at 137.16 101.6 0)
 		(mirror y)
@@
 	)
 	(symbol
-		(lib_id "power:GND")
+		(lib_id "gnd_NoFootPrint:GND")
 		(at 384.81 135.89 0)
 		(unit 1)
@@
 	)
 	(symbol
-		(lib_id "power:GND")
+		(lib_id "gnd_NoFootPrint:GND")
 		(at 381 105.41 0)
 		(unit 1)
@@
 	)
 	(symbol
-		(lib_id "power:GND")
+		(lib_id "gnd_NoFootPrint:GND")
 		(at 346.71 231.14 0)
 		(unit 1)
@@
 	)
 	(symbol
-		(lib_id "power:GND")
+		(lib_id "gnd_NoFootPrint:GND")
 		(at 436.88 147.32 0)
 		(unit 1)
@@
 	)
 	(symbol
-		(lib_id "power:GND")
+		(lib_id "gnd_NoFootPrint:GND")
 		(at 344.17 337.82 0)
 		(unit 1)
@@
 	)
 	(symbol
-		(lib_id "power:GND")
+		(lib_id "gnd_NoFootPrint:GND")
 		(at 309.88 67.31 0)
 		(unit 1)
@@
 	)
 	(symbol
-		(lib_id "power:GND")
+		(lib_id "gnd_NoFootPrint:GND")
 		(at 91.44 257.81 0)
 		(unit 1)
@@
 	)
 	(symbol
-		(lib_id "Interface_Expansion:TCA9535PWR")
+		(lib_id "Project_Parts:TCA9535PWR")
 		(at 204.47 245.11 0)
 		(unit 1)
@@
 	)
 	(symbol
-		(lib_id "power:GND")
+		(lib_id "gnd_NoFootPrint:GND")
 		(at 109.22 95.25 0)
 		(mirror y)
@@
 	)
 	(symbol
-		(lib_id "power:GND")
+		(lib_id "gnd_NoFootPrint:GND")
 		(at 406.4 223.52 0)
 		(unit 1)
@@
 	)
 	(symbol
-		(lib_id "power:GND")
+		(lib_id "gnd_NoFootPrint:GND")
 		(at 90.17 276.86 0)
 		(unit 1)
@@
 	)
 	(symbol
-		(lib_id "power:GND")
+		(lib_id "gnd_NoFootPrint:GND")
 		(at 330.2 337.82 0)
 		(unit 1)

Commit message: Bug fix
Parts:
- J2: symbol Connector:USB_C_Receptacle_USB2.0_16P -> Project_Parts:USB_C_Receptacle_USB2.0_16P
- J4: symbol Connector:Micro_SD_Card_Det_Hirose_DM3AT -> Project_Parts:Micro_SD_Card_Det_Hirose_DM3AT
- U14: symbol SamacSys_Parts:TPS3840DL30DBVR -> Project_Parts:TPS3840DL30DBVR
- U15: symbol Security:ATECC608B-SSHDA -> Project_Parts:ATECC608B-SSHDA
- U20: symbol SamacSys_Parts:W25N01GVZEIG -> Project_Parts:W25N01GVZEIG
- U23: symbol SamacSys_Parts:TPS22918TDBVTQ1 -> Project_Parts:TPS22918TDBVTQ1
- U903: symbol SN74AXC4T245QPWRQ1:SN74AXC4T245QPWRQ1 -> Project_Parts:SN74AXC4T245QPWRQ1_second
Changed lines of the file:
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@@
 	(wire
 		(pts
-			(xy 307.34 87.63) (xy 332.74 87.63)
+			(xy 307.34 87.63) (xy 344.17 87.63)
 		)
 		(stroke
@@
 	(wire
 		(pts
+			(xy 351.79 87.63) (xy 391.16 87.63)
+		)
+		(stroke
+			(width 0)
+			(type default)
+		)
+	)
+	(wire
+		(pts
 			(xy 128.27 210.82) (xy 161.29 210.82)
 		)
@@
 	(wire
 		(pts
-			(xy 340.36 87.63) (xy 394.97 87.63)
-		)
-		(stroke
-			(width 0)
-			(type default)
-		)
-	)
-	(wire
-		(pts
 			(xy 209.55 345.44) (xy 212.09 345.44)
 		)
@@
 		)
 	)
-	(label ""
-		(at 360.68 87.63 0)
-		(fields_autoplaced yes)
-		(effects
-			(font
-				(size 1.27 1.27)
-			)
-			(justify left bottom)
-		)
-		(property "GNSS" ""
-			(at 360.68 88.9 0)
-			(show_name no)
-			(do_not_autoplace no)
-			(effects
-				(font
-					(size 1.27 1.27)
-					(italic yes)
-				)
-				(justify left)
-			)
-		)
-	)
 	(label "SPI_SCLK"
 		(at 313.69 361.95 180)
@@
 	(global_label "GNSS_UART_TX"
 		(shape output)
-		(at 394.97 87.63 0)
+		(at 391.16 87.63 0)
 		(fields_autoplaced yes)
 		(effects
@@
 		)
 		(property "Intersheetrefs" "${INTERSHEET_REFS}"
-			(at 411.7437 87.63 0)
+			(at 407.9337 87.63 0)
 			(hide yes)
 			(show_name no)
@@
 	)
 	(symbol
-		(lib_id "Connector:Micro_SD_Card_Det_Hirose_DM3AT")
+		(lib_id "Project_Parts:Micro_SD_Card_Det_Hirose_DM3AT")
 		(at 485.14 257.81 0)
 		(unit 1)
@@
 	)
 	(symbol
-		(lib_id "SamacSys_Parts:TPS22918TDBVTQ1")
+		(lib_id "Project_Parts:TPS22918TDBVTQ1")
 		(at 463.55 205.74 0)
 		(unit 1)
@@
 	(symbol
 		(lib_id "Device:R")
+		(at 347.98 87.63 90)
+		(unit 1)
+		(body_style 1)
+		(exclude_from_sim no)
+		(in_bom yes)
+		(on_board yes)
+		(in_pos_files yes)
+		(dnp no)
+		(property "Reference" "R205"
+			(at 346.202 89.916 90)
+			(show_name no)
+			(do_not_autoplace no)
+			(effects
+				(font
+					(size 1.27 1.27)
+				)
+				(justify right)
+			)
+		)
+		(property "Value" "499"
+			(at 346.202 87.63 90)
+			(show_name no)
+			(do_not_autoplace no)
+			(effects
+				(font
+					(size 1.27 1.27)
+				)
+				(justify right)
+			)
+		)
+		(property "Footprint" "Resistor_SMD:R_0603_1608Metric"
+			(at 347.98 89.408 90)
+			(hide yes)
+			(show_name no)
+			(do_not_autoplace no)
+			(effects
+				(font
+					(size 1.27 1.27)
+				)
+			)
+		)
+		(property "Datasheet" ""
+			(at 347.98 87.63 0)
+			(hide yes)
+			(show_name no)
+			(do_not_autoplace no)
+			(effects
+				(font
+					(size 1.27 1.27)
+				)
+			)
+		)
+		(property "Description" "Resistor"
+			(at 347.98 87.63 0)
+			(hide yes)
+			(show_name no)
+			(do_not_autoplace no)
+			(effects
+				(font
+					(size 1.27 1.27)
+				)
+			)
+		)
+		(pin "1"
+		)
+		(pin "2"
+		)
+		(instances
+			(project "Tracker"
+				(path "/586d1ea1-b017-4713-987c-545d658f6cc8/378094db-8f3e-4510-9f4d-07bbb8577682"
+					(reference "R205")
+					(unit 1)
+				)
+			)
+		)
+	)
+	(symbol
+		(lib_id "Device:R")
 		(at 245.11 210.82 180)
 		(unit 1)
@@
 	)
 	(symbol
-		(lib_id "Connector:USB_C_Receptacle_USB2.0_16P")
+		(lib_id "Project_Parts:USB_C_Receptacle_USB2.0_16P")
 		(at 45.72 274.32 0)
 		(unit 1)
@@
 	)
 	(symbol
-		(lib_name "SN74AXC4T245QPWRQ1_1")
-		(lib_id "SN74AXC4T245QPWRQ1:SN74AXC4T245QPWRQ1")
+		(lib_id "Project_Parts:SN74AXC4T245QPWRQ1_second")
 		(at 346.71 273.05 0)
 		(unit 1)
@@
 	)
 	(symbol
-		(lib_id "Security:ATECC608B-SSHDA")
+		(lib_id "Project_Parts:ATECC608B-SSHDA")
 		(at 120.65 208.28 0)
 		(unit 1)
@@
 	(symbol
 		(lib_id "Device:R")
-		(at 336.55 87.63 90)
-		(unit 1)
-		(body_style 1)
-		(exclude_from_sim no)
-		(in_bom yes)
-		(on_board yes)
-		(in_pos_files yes)
-		(dnp no)
-		(property "Reference" "R205"
-			(at 334.772 89.916 90)
-			(show_name no)
-			(do_not_autoplace no)
-			(effects
-				(font
-					(size 1.27 1.27)
-				)
-				(justify right)
-			)
-		)
-		(property "Value" "499"
-			(at 334.772 87.63 90)
-			(show_name no)
-			(do_not_autoplace no)
-			(effects
-				(font
-					(size 1.27 1.27)
-				)
-				(justify right)
-			)
-		)
-		(property "Footprint" "Resistor_SMD:R_0603_1608Metric"
-			(at 336.55 89.408 90)
-			(hide yes)
-			(show_name no)
-			(do_not_autoplace no)
-			(effects
-				(font
-					(size 1.27 1.27)
-				)
-			)
-		)
-		(property "Datasheet" ""
-			(at 336.55 87.63 0)
-			(hide yes)
-			(show_name no)
-			(do_not_autoplace no)
-			(effects
-				(font
-					(size 1.27 1.27)
-				)
-			)
-		)
-		(property "Description" "Resistor"
-			(at 336.55 87.63 0)
-			(hide yes)
-			(show_name no)
-			(do_not_autoplace no)
-			(effects
-				(font
-					(size 1.27 1.27)
-				)
-			)
-		)
-		(pin "1"
-		)
-		(pin "2"
-		)
-		(instances
-			(project "Tracker"
-				(path "/586d1ea1-b017-4713-987c-545d658f6cc8/378094db-8f3e-4510-9f4d-07bbb8577682"
-					(reference "R205")
-					(unit 1)
-				)
-			)
-		)
-	)
-	(symbol
-		(lib_id "Device:R")
 		(at 90.17 273.05 0)
 		(unit 1)
@@
 	)
 	(symbol
-		(lib_id "SamacSys_Parts:TPS3840DL30DBVR")
+		(lib_id "Project_Parts:TPS3840DL30DBVR")
 		(at 73.66 87.63 0)
 		(unit 1)
@@
 	)
 	(symbol
-		(lib_id "SamacSys_Parts:W25N01GVZEIG")
+		(lib_id "Project_Parts:W25N01GVZEIG")
 		(at 336.55 355.6 0)
 		(unit 1)

Commit message: bug
Parts:
- J4: symbol Project_Parts:Micro_SD_Card_Det_Hirose_DM3AT -> Project_Parts:Micro_SD_Card_Det_Hirose_DM3AT_new
Connections:
- net GND: now also J4.11 (SHIELD); no longer J4.SH (SHIELD)
Changed lines of the file:
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@@
 	)
 	(symbol
-		(lib_id "Project_Parts:Micro_SD_Card_Det_Hirose_DM3AT")
+		(lib_id "Project_Parts:Micro_SD_Card_Det_Hirose_DM3AT_new")
 		(at 485.14 257.81 0)
 		(unit 1)
@@
 		(pin "7"
 		)
-		(pin "SH"
+		(pin "11"
 		)
 		(pin "1"

Commit message: Bug
Parts:
- J4: symbol Project_Parts:Micro_SD_Card_Det_Hirose_DM3AT_new -> Project_Parts:Micro_SD_Card_Det_Hirose_DM3AT_SH
Connections:
- net GND: now also J4.SH (SHIELD); no longer J4.11 (SHIELD)
Changed lines of the file:
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@@
 	)
 	(symbol
-		(lib_id "Project_Parts:Micro_SD_Card_Det_Hirose_DM3AT_new")
+		(lib_id "Project_Parts:Micro_SD_Card_Det_Hirose_DM3AT_SH")
 		(at 485.14 257.81 0)
 		(unit 1)
@@
 		(pin "7"
 		)
-		(pin "11"
+		(pin "SH"
 		)
 		(pin "1"

Commit message: updt
Parts:
- removed C61, C62, C63: DNP, Capacitor_SMD:C_0402_1005Metric, symbol Device:C
- removed R49: DNP, Resistor_SMD:R_0603_1608Metric, symbol Device:R
- removed R50, R52: 10k, Resistor_SMD:R_0603_1608Metric, symbol Device:R
- removed R801: 10k, Resistor_SMD:R_0402_1005Metric, symbol Device:R
- C44: value 100nF -> 10nF
- C48: value 10uF 10V -> 4.7uF 10V
Connections:
- net CAN1_RXD: no longer names the net of U19.23 (CAN_RX+strap(GPIO15))
- net CAN1_TXD: no longer names the net of U19.10 (CAN-TX+bootstrap(GPIO8))
- net TEMP_ALERT_N: no longer names the net of U802.3 (ALERT)
- no-connect marks 0 -> 3
