File: Tracker.kicad_sch (KiCad schematic)
At the start: 140 parts, among them J1 Vehicle 12V 2X2, J303 Conn_Coaxial, Q1 DMT6007LFGQ-7, Q10 2N7002, Q2 2N7002, Q4 CSD16406Q3, Q5 CSD16406Q3, U1 LM74700, U10 TPS62840DLCR, U11 TPS62840DLCR, U2 LM76003QRNPRQ1, U3 TPS2121RUXR, U305 MAX-M10S, U4 INA3221AIRGVR, U5 BQ25601DRTWR, U6 BQ29700DSER, U7 TPS3840DL35DBVR, U8 TPS63802DLAR, U9 TPS61094DSSR

Commit message: Footprint
Parts:
- BT1: footprint BHC186501P -> SamacSys_Parts:BHC186501P
- C19, C20, C21: footprint (none) -> Capacitor_SMD:C_0603_1608Metric
- C22: footprint (none) -> Capacitor_SMD:C_0805_2012Metric
- C30, C31, C32, C33, C34, C35, C36, C37, C38, C39, C40, C41, C42, C43, C45, C46, C47, CSC1, U4: footprint QFN65P400X400X100-17N-D -> SamacSys_Parts:QFN65P400X400X100-17N-D
- D2, U5: footprint QFN50P400X400X80-25N-D -> SamacSys_Parts:QFN50P400X400X80-25N-D
- D3: footprint DIONM5436X244N -> SamacSys_Parts:DIONM5436X244N
- F1: value 3A -> 3A slow-blow, 125V; footprint (none) -> Fuse:Fuse_Littelfuse-NANO2-451_453
- L2: footprint (none) -> Inductor_SMD:L_Coilcraft_XAL6030-XXX
- Q1: footprint DMTH8008LFGQ7 -> SamacSys_Parts:DMTH8008LFGQ7
- Q4, Q5: footprint DQG_VSON-CLIP -> SamacSys_Parts:DQG_VSON-CLIP
- R1, R28, R3, R323: footprint (none) -> Resistor_SMD:R_1206_3216Metric
- R10, R11, R2, R23, R26, R27, R29, R31, R316, R32, R321, R322, R33, R4, R40, R42, R43, R44, R45, R46, R6, R7, R70, R8, R9: footprint (none) -> Resistor_SMD:R_0603_1608Metric
- R13, R14, R15, R16, R17, R18, R19, R21, R35, R36, R37, U3: footprint TPS2121RUXR -> SamacSys_Parts:TPS2121RUXR
- R313: footprint (none) -> Resistor_SMD:R_0402_1005Metric
- R39: footprint (none) -> Rotary_Encoder:RotaryEncoder_Bourns_Horizontal_PEL12D-2x18F-Sxxxx
- R47: footprint TPS2121RUXR -> Resistor_SMD:R_0603_1608Metric
- TP1: footprint DMTH8008LFGQ7 -> TestPoint:TestPoint_Pad_D1.5mm
- TP10, TP11, TP208, TP3, TP9: footprint (none) -> TestPoint:TestPoint_Pad_D1.5mm
- TP309, TP310, TP311: footprint RF_GPS:ublox_MAX -> TestPoint:TestPoint_Pad_D1.5mm
- TP4, TP5, TP6: footprint Relay_THT:Relay_DPDT_Schrack-RT2-FormC_RM5mm -> TestPoint:TestPoint_Pad_D1.5mm
- TP7, TP8: footprint SOT95P280X145-5N -> TestPoint:TestPoint_Pad_D1.5mm
- U10, U11: footprint SON50P150X200X100-8N-D -> SamacSys_Parts:SON50P150X200X100-8N-D
- U2: footprint LM76003QRNPRQ1 -> SamacSys_Parts:LM76003QRNPRQ1
- U6: footprint SON50P150X150X80-6N -> SamacSys_Parts:SON50P150X150X80-6N
- U7: footprint SOT95P280X145-5N -> SamacSys_Parts:SOT95P280X145-5N
- U8: footprint TPS63802DLAR -> SamacSys_Parts:TPS63802DLAR
- U9: footprint SON50P200X300X80-13N-D -> SamacSys_Parts:SON50P200X300X80-13N-D
Connections:
- net BG95_PG: now reaches R47.1, TP208.1, U8.5 (PG)

Commit message: Footprint
Parts:
- C1, C10, C12, C13, C14, C15, C2, C23, C3, C321, C4, C5: footprint Package_SO:SOIC-8_3.9x4.9mm_P1.27mm -> Capacitor_SMD:C_0603_1608Metric
- C11: footprint Package_SO:SOIC-8_3.9x4.9mm_P1.27mm -> Capacitor_SMD:CP_Elec_8x10.5
- C16, C17, C18, C6, C7, C8, C9: footprint Package_SO:SOIC-8_3.9x4.9mm_P1.27mm -> Capacitor_SMD:C_1210_3225Metric
- C24: footprint Package_SO:SOIC-8_3.9x4.9mm_P1.27mm -> Capacitor_SMD:C_1206_3216Metric
- C25, C26, C27, C28: footprint Package_SO:SOIC-8_3.9x4.9mm_P1.27mm -> Capacitor_SMD:C_0805_2012Metric
- C30, C31, C42, C43, C45, C46: footprint SamacSys_Parts:QFN65P400X400X100-17N-D -> Capacitor_SMD:C_0603_1608Metric
- C316: footprint RF_Module:ESP32-C6-MINI-1 -> Capacitor_SMD:C_0402_1005Metric
- C322, C323: footprint Package_SO:SOIC-8_3.9x4.9mm_P1.27mm -> Capacitor_SMD:C_0402_1005Metric
- C33, C34, C35, C37, C38, C39, C40, C41, C47: footprint SamacSys_Parts:QFN65P400X400X100-17N-D -> Capacitor_SMD:C_0805_2012Metric
- C36: footprint SamacSys_Parts:QFN65P400X400X100-17N-D -> Capacitor_Tantalum_SMD:CP_EIA-7343-31_Kemet-D
- CSC1: footprint SamacSys_Parts:QFN65P400X400X100-17N-D -> Capacitor_THT:CP_Radial_D8.0mm_P3.50mm
- D2: footprint SamacSys_Parts:QFN50P400X400X80-25N-D -> LED_SMD:LED_0603_1608Metric
- J1: footprint Package_TO_SOT_SMD:SOT-23 -> Connector_Molex:Molex_Micro-Fit_3.0_43045-0400_2x02_P3.00mm_Horizontal
- J303: footprint Package_DFN_QFN:WDFN-10-1EP_3x3mm_P0.5mm_EP1.8x2.5mm -> Connector_Coaxial:U.FL_Hirose_U.FL-R-SMT-1_Vertical
- L4: footprint Relay_THT:Relay_DPDT_Finder_30.22 -> Inductor_SMD:L_Coilcraft_XFL2010
- R13, R14, R15, R16, R17, R18, R19, R35, R36, R37: footprint SamacSys_Parts:TPS2121RUXR -> Resistor_SMD:R_0603_1608Metric
- R21: footprint SamacSys_Parts:TPS2121RUXR -> Resistor_SMD:R_1206_3216Metric
- R39: footprint Rotary_Encoder:RotaryEncoder_Bourns_Horizontal_PEL12D-2x18F-Sxxxx -> Resistor_SMD:R_0603_1608Metric
- TH1: footprint Resistor_THT:R_Array_SIP4 -> Resistor_THT:R_Axial_DIN0204_L3.6mm_D1.6mm_P5.08mm_Horizontal

Commit message: Update fix
Parts:
- BT1: symbol SamacSys_Parts:BHC-18650-1P -> Project_Parts:BHC-18650-1P
- Q10, Q2: symbol Transistor_FET:2N7002 -> Project_Parts:2N7002
- U1: symbol Power_Management:LM74700 -> Project_Parts:LM74700
- U3: symbol SamacSys_Parts:TPS2121RUXR -> Project_Parts:TPS2121RUXR
- U6: symbol SamacSys_Parts:BQ29700DSER -> Project_Parts:BQ29700DSER
- U8: symbol SamacSys_Parts:TPS63802DLAR -> Project_Parts:TPS63802DLAR
- U9: symbol SamacSys_Parts:TPS61094DSSR -> Project_Parts:TPS61094DSSR

Commit message: Bug fix
Parts:
- D3: symbol SamacSys_Parts:SMBJ33CA -> Project_Parts:SMBJ33CA
- Q1: symbol SamacSys_Parts:DMT6007LFGQ-7 -> Project_Parts:DMT6007LFGQ-7
- Q4: symbol SamacSys_Parts:CSD16406Q3 -> Project_Parts:CSD16406Q3_Q4
- Q5: symbol SamacSys_Parts:CSD16406Q3 -> Project_Parts:CSD16406Q3_Q5
- U10: symbol SamacSys_Parts:TPS62840DLCR -> Project_Parts:TPS62840DLCR_U10
- U11: symbol SamacSys_Parts:TPS62840DLCR -> Project_Parts:TPS62840DLCR_U11
- U2: symbol SamacSys_Parts:LM76003QRNPRQ1 -> Project_Parts:LM76003QRNPRQ1
- U305: symbol RF_GPS:MAX-M10S -> Project_Parts:MAX-M10S
- U4: symbol SamacSys_Parts:INA3221AIRGVR -> Project_Parts:INA3221AIRGVR
- U5: symbol SamacSys_Parts:BQ25601DRTWR -> Project_Parts:BQ25601DRTWR
- U7: symbol SamacSys_Parts:TPS3840DL35DBVR -> Project_Parts:TPS3840DL35DBVR
Other:
- moved on the sheet: C19, C20, C21, C22, R13, R14, R15, R16, R17, R18, R19, R21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

Commit message: bug
Parts:
- C29: footprint Package_SO:SOIC-8_3.9x4.9mm_P1.27mm -> Capacitor_SMD:C_0805_2012Metric
- C32: footprint SamacSys_Parts:QFN65P400X400X100-17N-D -> Capacitor_SMD:C_0603_1608Metric
- L1, L3: footprint Relay_THT:Relay_DPDT_Finder_30.22 -> Inductor_SMD:L_Coilcraft_XAL5030-XXX
- L301: footprint Relay_THT:Relay_DPDT_Finder_30.22 -> Inductor_SMD:L_0402_1005Metric
- L7, L8: footprint Relay_THT:Relay_DPDT_Finder_30.22 -> Inductor_SMD:L_Murata_DFE201610P
Changed lines of the file:
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@@
 			)
 		)
-		(property "Footprint" "Relay_THT:Relay_DPDT_Finder_30.22"
+		(property "Footprint" "Inductor_SMD:L_Murata_DFE201610P"
 			(at 278.13 48.26 0)
 			(hide yes)
@@
 			)
 		)
-		(property "Footprint" "Relay_THT:Relay_DPDT_Finder_30.22"
+		(property "Footprint" "Inductor_SMD:L_0402_1005Metric"
 			(at 490.22 262.89 0)
 			(hide yes)
@@
 			)
 		)
-		(property "Footprint" "SamacSys_Parts:QFN65P400X400X100-17N-D"
+		(property "Footprint" "Capacitor_SMD:C_0603_1608Metric"
 			(at 228.2952 201.93 0)
 			(hide yes)
@@
 			)
 		)
-		(property "Footprint" "Relay_THT:Relay_DPDT_Finder_30.22"
+		(property "Footprint" "Inductor_SMD:L_Coilcraft_XAL5030-XXX"
 			(at 367.03 147.32 0)
 			(hide yes)
@@
 			)
 		)
-		(property "Footprint" "Relay_THT:Relay_DPDT_Finder_30.22"
+		(property "Footprint" "Inductor_SMD:L_Murata_DFE201610P"
 			(at 279.4 83.82 0)
 			(hide yes)
@@
 			)
 		)
-		(property "Footprint" "Relay_THT:Relay_DPDT_Finder_30.22"
+		(property "Footprint" "Inductor_SMD:L_Coilcraft_XAL5030-XXX"
 			(at 332.74 241.3 0)
 			(hide yes)
@@
 			)
 		)
-		(property "Footprint" "Package_SO:SOIC-8_3.9x4.9mm_P1.27mm"
+		(property "Footprint" "Capacitor_SMD:C_0805_2012Metric"
 			(at 345.1352 283.21 0)
 			(hide yes)

Commit message: Bug
Parts:
- L4: footprint Inductor_SMD:L_Coilcraft_XFL2010 -> TI_Parts:IND_XGL4020_COC
- L5: footprint Relay_THT:Relay_DPDT_Finder_30.22 -> TI_Parts:IND_XGL4020_COC
Changed lines of the file:
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@@
 			)
 		)
-		(property "Footprint" "Inductor_SMD:L_Coilcraft_XFL2010"
+		(property "Footprint" "TI_Parts:IND_XGL4020_COC"
 			(at 110.49 72.39 0)
 			(hide yes)
@@
 			)
 		)
-		(property "Footprint" "Relay_THT:Relay_DPDT_Finder_30.22"
+		(property "Footprint" "TI_Parts:IND_XGL4020_COC"
 			(at 86.36 260.35 0)
 			(hide yes)

Commit message: update
Parts:
- L4: value 0.47uH 5.4A -> 0.47uH XGL4020-471MEC; MPN (none) -> XGL4020-471MEC; Manufacturer (none) -> Coilcraft
- L5: value 2.2uH 4.4A -> 2.2uH XGL4020-222MEC; MPN (none) -> XGL4020-222MEC; Manufacturer (none) -> Coilcraft
Changed lines of the file:
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@@
 			)
 		)
-		(property "Value" "0.47uH 5.4A"
+		(property "Value" "0.47uH XGL4020-471MEC"
 			(at 110.49 69.85 90)
 			(show_name no)
@@
 		(property "Description" "Inductor"
 			(at 110.49 72.39 0)
+			(hide yes)
+			(show_name no)
+			(do_not_autoplace no)
+			(effects
+				(font
+					(size 1.27 1.27)
+				)
+			)
+		)
+		(property "MPN" "XGL4020-471MEC"
+			(at 110.49 72.39 90)
+			(hide yes)
+			(show_name no)
+			(do_not_autoplace no)
+			(effects
+				(font
+					(size 1.27 1.27)
+				)
+			)
+		)
+		(property "Manufacturer" "Coilcraft"
+			(at 110.49 72.39 90)
 			(hide yes)
 			(show_name no)
@@
 			)
 		)
-		(property "Value" "2.2uH 4.4A"
+		(property "Value" "2.2uH XGL4020-222MEC"
 			(at 79.756 261.112 0)
 			(show_name no)
@@
 			(at 86.36 260.35 0)
 			(hide yes)
+			(show_name no)
+			(do_not_autoplace no)
+			(effects
+				(font
+					(size 1.27 1.27)
+				)
+			)
+		)
+		(property "MPN" "XGL4020-222MEC"
+			(at 86.36 260.35 0)
+			(hide yes)
+			(show_name no)
+			(do_not_autoplace no)
+			(effects
+				(font
+					(size 1.27 1.27)
+				)
+			)
+		)
+		(property "Manufacturer" "Coilcraft"
+			(at 86.36 260.35 0)
+			(hide yes)

Commit message: updt
Parts:
- removed R47: 100k, Resistor_SMD:R_0603_1608Metric, symbol Device:R
Changed lines of the file:
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@@
 	)
 	(junction
-		(at 83.82 88.9)
-		(diameter 0)
-		(color 0 0 0 0)
-	)
-	(junction
 		(at 441.96 149.86)
 		(diameter 0)
@@
 	(wire
 		(pts
-			(xy 83.82 88.9) (xy 86.36 88.9)
+			(xy 76.2 88.9) (xy 86.36 88.9)
 		)
 		(stroke
@@
 	(wire
 		(pts
-			(xy 76.2 88.9) (xy 83.82 88.9)
-		)
-		(stroke
-			(width 0)
-			(type default)
-		)
-	)
-	(wire
-		(pts
 			(xy 113.03 140.97) (xy 114.3 140.97)
 		)
@@
 	(wire
 		(pts
-			(xy 83.82 93.98) (xy 83.82 88.9)
-		)
-		(stroke
-			(width 0)
-			(type default)
-		)
-	)
-	(wire
-		(pts
 			(xy 299.72 83.82) (xy 299.72 81.28)
 		)
@@
 	(wire
 		(pts
-			(xy 83.82 101.6) (xy 83.82 104.14)
-		)
-		(stroke
-			(width 0)
-			(type default)
-		)
-	)
-	(wire
-		(pts
 			(xy 373.38 154.94) (xy 355.6 154.94)
 		)
@@
 	)
 	(symbol
-		(lib_id "power:VCC")
-		(at 83.82 104.14 270)
-		(unit 1)
-		(body_style 1)
-		(exclude_from_sim no)
-		(in_bom yes)
-		(on_board yes)
-		(in_pos_files yes)
-		(dnp no)
-		(fields_autoplaced yes)
-		(property "Reference" "#PWR0171"
-			(at 80.01 104.14 0)
-			(hide yes)
-			(show_name no)
-			(do_not_autoplace no)
-			(effects
-				(font
-					(size 1.27 1.27)
-				)
-			)
-		)
-		(property "Value" "3V3_AON"
-			(at 87.63 104.1399 90)
-			(show_name no)
-			(do_not_autoplace no)
-			(effects
-				(font
-					(size 1.27 1.27)
-				)
-				(justify left)
-			)
-		)
-		(property "Footprint" "Package_QFP:TQFP-44_10x10mm_P0.8mm"
-			(at 83.82 104.14 0)
-			(hide yes)
-			(show_name no)
-			(do_not_autoplace no)
-			(effects
-				(font
-					(size 1.27 1.27)
-				)
-			)
-		)
-		(property "Datasheet" ""
-			(at 83.82 104.14 0)
-			(hide yes)
-			(show_name no)
-			(do_not_autoplace no)
-			(effects
-				(font
-					(size 1.27 1.27)
-				)
-			)
-		)
-		(property "Description" "Power symbol creates a global label with name \"VCC\""
-			(at 83.82 104.14 0)
-			(hide yes)
-			(show_name no)
-			(do_not_autoplace no)
-			(effects
-				(font
-					(size 1.27 1.27)
-				)
-			)
-		)
-		(pin "1"
-		)
-		(instances
-			(project "Tracker"
-				(path "/586d1ea1-b017-4713-987c-545d658f6cc8"
-					(reference "#PWR0171")
-					(unit 1)
-				)
-			)
-		)
-	)
-	(symbol
 		(lib_id "power:PWR_FLAG")
 		(at 229.87 345.44 0)
@@
 					(unit 1)
 				)
-			)
-		)
-	)
-	(symbol
-		(lib_id "Device:R")
-		(at 83.82 97.79 0)
-		(unit 1)
-		(body_style 1)
-		(exclude_from_sim no)
-		(in_bom yes)
-		(on_board yes)
-		(in_pos_files yes)
-		(dnp no)
-		(property "Reference" "R47"
-			(at 77.978 97.79 0)
-			(show_name no)
-			(do_not_autoplace no)
-			(effects
-				(font
-					(size 1.27 1.27)
-				)
-				(justify left)
-			)
-		)
-		(property "Value" "100k"
-			(at 77.216 99.568 0)
-			(show_name no)
-			(do_not_autoplace no)
-			(effects
-				(font
-					(size 1.27 1.27)
-				)
-				(justify left)
-			)
-		)
-		(property "Footprint" "Resistor_SMD:R_0603_1608Metric"
-			(at 82.042 97.79 90)
-			(hide yes)
-			(show_name no)
-			(do_not_autoplace no)
-			(effects
-				(font
-					(size 1.27 1.27)
-				)
-			)
-		)
-		(property "Datasheet" ""
-			(at 83.82 97.79 0)
-			(hide yes)
-			(show_name no)
-			(do_not_autoplace no)
-			(effects
-				(font
-					(size 1.27 1.27)
-				)
-			)
-		)
-		(property "Description" "Resistor"
-			(at 83.82 97.79 0)
-			(hide yes)
-			(show_name no)
-			(do_not_autoplace no)
-			(effects
-				(font
-					(size 1.27 1.27)
-				)
-			)
-		)
-		(pin "1"
-		)
-		(pin "2"
-		)
-		(instances
-			(project "Tracker"
-				(path "/586d1ea1-b017-4713-987c-545d658f6cc8"
-					(reference "R47")
-					(unit 1)
-				)
