File: Tracker.kicad_sch (KiCad schematic)
At the start: 139 parts, among them J1 Vehicle 12V 2X2, J303 Conn_Coaxial, Q1 DMT6007LFGQ-7, Q10 2N7002, Q2 2N7002, Q4 CSD16406Q3, Q5 CSD16406Q3, U1 LM74700, U10 TPS62840DLCR, U11 TPS62840DLCR, U2 LM76003QRNPRQ1, U3 TPS2121RUXR, U305 MAX-M10S, U4 INA3221AIRGVR, U5 BQ25601DRTWR, U6 BQ29700DSER, U7 TPS3840DL35DBVR, U8 TPS63802DLAR, U9 TPS61094DSSR

Commit message: update
Parts:
- renumbered C20 to C1, C22 to C10, C35 to C11, C21 to C12, C40 to C13, C36 to C14, C41 to C15, C45 to C16, C30 to C17, C43 to C18, C32 to C19, C42 to C2, C23 to C20, C24 to C21, C47 to C22, C46 to C23, C25 to C24, C6 to C25, C29 to C27, C7 to C28, C28 to C29, C33 to C3, C27 to C30, C8 to C31, C9 to C32, C5 to C33, C10 to C34, C11 to C35, C1 to C36, C13 to C37, C322 to C38, C14 to C39, C37 to C4, C2 to C40, C321 to C41, C323 to C42, C3 to C43, C12 to C44, C316 to C45, C18 to C46, C4 to C47, C15 to C48, C17 to C49, C38 to C5, C16 to C50, C31 to C6, C19 to C7, C34 to C8, C39 to C9, D2 to D1, D3 to D2, J303 to J2, L5 to L1, L4 to L2, L8 to L3, L7 to L4, L3 to L5, L1 to L6, L301 to L7, L2 to L8, Q4 to Q1, Q5 to Q2, Q10 to Q3, Q2 to Q4, Q1 to Q5, R42 to R1, R36 to R10, R39 to R11, R29 to R12, R17 to R13, R18 to R14, R40 to R15, R31 to R16, R32 to R17, R21 to R18, R33 to R19, R43 to R2, R44 to R20, R46 to R21, R27 to R22, R26 to R23, R70 to R24, R45 to R25, R23 to R26, R322 to R27, R321 to R28, R323 to R29, R15 to R3, R28 to R30, R3 to R31, R4 to R32, R316 to R33, R7 to R34, R6 to R35, R10 to R36, R11 to R37, R313 to R38, R9 to R39, R16 to R4, R1 to R40, R2 to R41, R8 to R42, R37 to R5, R13 to R6, R14 to R7, R19 to R8, R35 to R9, TP208 to TP1, TP311 to TP10, TP310 to TP11, TP309 to TP12, TP1 to TP13, TP7 to TP14, TP3 to TP2, TP8 to TP3, TP9 to TP4, TP4 to TP5, TP10 to TP6, TP11 to TP7, TP6 to TP8, TP5 to TP9, U3 to U1, U2 to U10, U305 to U11, U1 to U12, U8 to U2, U9 to U3, U6 to U4, U4 to U5, U7 to U6, U10 to U7, U11 to U8, U5 to U9

Commit message: BT1 update
Parts:
- BT1: footprint SamacSys_Parts:BHC186501P -> Battery:BatteryHolder_MPD_BH-18650-PC
Changed lines of the file:
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@@
 			)
 		)
-		(property "Footprint" "SamacSys_Parts:BHC186501P"
+		(property "Footprint" "Battery:BatteryHolder_MPD_BH-18650-PC"
 			(at 68.58 425.12 0)
 			(hide yes)

Commit message: Fix
Parts:
- removed BT1: BHC-18650-1P, Battery:BatteryHolder_MPD_BH-18650-PC, symbol Project_Parts:BHC-18650-1P
- removed C35: 47uF 100V, Capacitor_SMD:CP_Elec_8x10.5, symbol Device:C
- added BT2: BH-18650-PC, Battery:BatteryHolder_MPD_BH-18650-PC, symbol BH-18650-PC:BH-18650-PC
- added C35: 47uF 100V, Capacitor_SMD:CP_Elec_8x10.5, symbol Device:C_Polarized
Connections:
- net BAT_CELL: now also BT2.P
- net GND: now also C35.2
- net at C31.2, C32.2, C34.2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: now also C35.1
- net at C6.2, Q1.1 (S_1), Q1.2 (S_2)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: now also BT2.N

Commit message: fix
Changed lines of the file:
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@@
 	)
 	(junction
-		(at 49.53 326.39)
+		(at 52.07 326.39)
 		(diameter 0)
 		(color 0 0 0 0)
@@
 	(wire
 		(pts
-			(xy 49.53 326.39) (xy 87.63 326.39)
-		)
-		(stroke
-			(width 0)
-			(type default)
-		)
-	)
-	(wire
-		(pts
 			(xy 388.62 147.32) (xy 417.83 147.32)
 		)
@@
 	(wire
 		(pts
-			(xy 49.53 326.39) (xy 49.53 327.66)
+			(xy 52.07 326.39) (xy 52.07 328.93)
 		)
 		(stroke
@@
 	(wire
 		(pts
-			(xy 45.72 326.39) (xy 49.53 326.39)
+			(xy 45.72 326.39) (xy 87.63 326.39)
 		)
 		(stroke
@@
 	(wire
 		(pts
-			(xy 49.53 344.17) (xy 87.63 344.17)
+			(xy 52.07 344.17) (xy 87.63 344.17)
 		)
 		(stroke
@@
 	(wire
 		(pts
-			(xy 49.53 340.36) (xy 49.53 344.17)
+			(xy 52.07 341.63) (xy 52.07 344.17)
 		)
 		(stroke
@@
 	(symbol
 		(lib_id "BH-18650-PC:BH-18650-PC")
-		(at 49.53 335.28 270)
+		(at 52.07 336.55 270)
 		(unit 1)
 		(body_style 1)
@@
 		(fields_autoplaced yes)
 		(property "Reference" "BT2"
-			(at 53.34 331.4699 90)
+			(at 55.88 332.7399 90)
 			(hide yes)
 			(show_name no)
@@
 		)
 		(property "Value" "BH-18650-PC"
-			(at 53.34 334.0099 90)
+			(at 55.88 335.2799 90)
 			(hide yes)
 			(show_name no)
@@
 		)
 		(property "Footprint" "Battery:BatteryHolder_MPD_BH-18650-PC"
-			(at 49.53 335.28 0)
+			(at 52.07 336.55 0)
 			(hide yes)
 			(show_name no)
@@
 		)
 		(property "Datasheet" ""
-			(at 49.53 335.28 0)
+			(at 52.07 336.55 0)
 			(hide yes)
 			(show_name no)
@@
 		)
 		(property "Description" "18650 cell battery holders,li-ion battery holders"
-			(at 49.53 335.28 0)
+			(at 52.07 336.55 0)
 			(hide yes)
 			(show_name no)
@@
 		)
 		(property "MF" "MPD (Memory Protection Devices)"
-			(at 49.53 335.28 0)
+			(at 52.07 336.55 0)
 			(hide yes)
 			(show_name no)
@@
 		)
 		(property "MAXIMUM_PACKAGE_HEIGHT" "21.31mm"
-			(at 49.53 335.28 0)
+			(at 52.07 336.55 0)
 			(hide yes)
 			(show_name no)
@@
 		)
 		(property "Package" "None"
-			(at 49.53 335.28 0)
+			(at 52.07 336.55 0)
 			(hide yes)
 			(show_name no)
@@
 		)
 		(property "Price" "None"
-			(at 49.53 335.28 0)
+			(at 52.07 336.55 0)
 			(hide yes)
 			(show_name no)
@@
 		)
 		(property "Check_prices" "https://www.snapeda.com/parts/BH-18650-PC/MPD/view-part/?ref=eda"
-			(at 49.53 335.28 0)
+			(at 52.07 336.55 0)
 			(hide yes)
 			(show_name no)
@@
 		)
 		(property "STANDARD" "Manufacturer Recommendation"
-			(at 49.53 335.28 0)
+			(at 52.07 336.55 0)
 			(hide yes)
 			(show_name no)
@@
 		)
 		(property "PARTREV" "05/17/19"
-			(at 49.53 335.28 0)
+			(at 52.07 336.55 0)
 			(hide yes)
 			(show_name no)
@@
 		)
 		(property "SnapEDA_Link" "https://www.snapeda.com/parts/BH-18650-PC/MPD/view-part/?ref=snap"
-			(at 49.53 335.28 0)
+			(at 52.07 336.55 0)
 			(hide yes)
 			(show_name no)
@@
 		)
 		(property "MP" "BH-18650-PC"
-			(at 49.53 335.28 0)
+			(at 52.07 336.55 0)
 			(hide yes)
 			(show_name no)
@@
 		)
 		(property "Availability" "In Stock"
-			(at 49.53 335.28 0)
+			(at 52.07 336.55 0)
 			(hide yes)
 			(show_name no)
@@
 		)
 		(property "MANUFACTURER" "MPD"
-			(at 49.53 335.28 0)
+			(at 52.07 336.55 0)
 			(hide yes)
 			(show_name no)

Commit message: updt
Parts:
- BT2: footprint Battery:BatteryHolder_MPD_BH-18650-PC -> SamacSys_Parts:BAT_BH-18650-PC
Changed lines of the file:
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@@
 			)
 		)
-		(property "Footprint" "Battery:BatteryHolder_MPD_BH-18650-PC"
+		(property "Footprint" "SamacSys_Parts:BAT_BH-18650-PC"
 			(at 52.07 336.55 0)
 			(hide yes)

Commit message: updt
Parts:
- added H1, H2, H3, H4: MountingHole_3.2mm_M3, MountingHole:MountingHole_3.2mm_M3, symbol Mechanical:MountingHole
