File: Tracker.kicad_pcb (KiCad board)
At the start: 2 copper layers, 282 parts, among them J1 Vehicle 12V 2X2, J2 USB_C_Receptacle_USB2.0_16P, J3 Conn_01x05, J303 Conn_Coaxial, J4 Micro_SD_Card_Det_Hirose_DM3AT, J5 SIM8060-6-1-14-00-A, J6 Conn_Coaxial, J7 Conn_Coaxial, Q1 DMT6007LFGQ-7, Q10 2N7002, Q2 2N7002, Q4 CSD16406Q3, Q5 CSD16406Q3, Q6 MMBT3904, Q7 MMBT3904, SW1 RESET, SW2 BOOT, U1 LM74700, U10 TPS62840DLCR, U11 TPS62840DLCR, U12 USBLC6-2SC6, U14 TPS3840DL30DBVR, U15 ATECC608B-SSHDA, U16 USBLC6-2SC6, U17 ASM330LHHTR, U18 TCA9535PWR, U2 LM76003QRNPRQ1, U20 W25N01GVZEIG, U23 TPS22918TDBVTQ1, U24 SN74AXC4T245QPWRQ1_CELL, U25 SN74AXC4T245QPWRQ1, U26 BG95-M3, U3 TPS2121RUXR, U305 MAX-M10S, U4 INA3221AIRGVR, U5 BQ25601DRTWR, U6 BQ29700DSER, U7 TPS3840DL35DBVR, U8 TPS63802DLAR, U802 TMP1075DGKR, U9 TPS61094DSSR, U902 SN74AXC4T245QPWRQ1, U903 SN74AXC4T245QPWRQ1

Commit message: Update Tracker.kicad_pcb
Parts:
- added REF**: MountingHole_3.2mm_M3, MountingHole:MountingHole_3.2mm_M3, F.Cu at (196.0, 166.0)
- added REF**: MountingHole_3.2mm_M3, MountingHole:MountingHole_3.2mm_M3, F.Cu at (196.0, 104.0)
- added REF**: MountingHole_3.2mm_M3, MountingHole:MountingHole_3.2mm_M3, F.Cu at (104.0, 104.0)
- added REF**: MountingHole_3.2mm_M3, MountingHole:MountingHole_3.2mm_M3, F.Cu at (104.0, 166.0)
- BT1: moved to B.Cu
- moved J303 929.3 mm to (-810.6, 97.9)
- moved R12 136.5 mm to (230.7, 33.5)
- moved R602 136.3 mm to (261.4, 54.2)
- moved R62 136.0 mm to (270.5, 56.3)
- moved R63 136.0 mm to (270.5, 58.3)
- moved R65 136.0 mm to (270.5, 62.3)
- moved R1 136.0 mm to (248.7, 2.19)
- moved R10 136.0 mm to (218.5, 7.15)
- moved R11 136.0 mm to (218.5, 9.66)
- moved R13 136.0 mm to (222.5, -12.9)
- moved R14 136.0 mm to (222.5, -10.4)
- moved R15 136.0 mm to (222.5, -7.91)
- moved R16 136.0 mm to (222.5, -5.40)
- moved R17 136.0 mm to (222.5, -2.89)
- moved R18 136.0 mm to (222.5, -0.38)
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Other:
- board outline added: 100 x 70 mm
- copper layers 2 -> 4

Commit message: PCB
Parts:
- moved C10 227.4 mm to (186.3, 125.0)
- moved C12 221.8 mm to (176.8, 135.5)
- moved C15 218.0 mm to (176.8, 133.5)
- moved C1 214.0 mm to (174.7, 105.0), turned to 180 degrees
- moved C3 213.2 mm to (174.8, 107.5), turned to 180 degrees
- moved C4 213.1 mm to (174.7, 110.0), turned to 180 degrees
- moved C2 212.3 mm to (174.7, 102.5), turned to 180 degrees
- moved C31 205.2 mm to (149.5, 155.5), turned to 90 degrees
- moved C53 200.7 mm to (181.7, 149.0), turned to 180 degrees
- moved R31 186.4 mm to (145.5, 157.5)
- moved R33 186.4 mm to (145.5, 162.5)
- moved R63 172.1 mm to (132.0, 160.5)
- moved R53 167.2 mm to (106.5, 132.5)
- moved R801 166.5 mm to (116.0, 144.0)
- moved R32 164.2 mm to (145.5, 160.0), turned to 180 degrees
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
Commit message: updt
Parts:
- moved C29 181.6 mm to (157.5, 133.1), turned to 90 degrees
- moved C28 180.5 mm to (154.5, 133.0), turned to 90 degrees
- moved C27 179.5 mm to (151.5, 133.1), turned to 90 degrees
- moved C26 178.6 mm to (148.5, 133.1), turned to 90 degrees
- moved C25 177.7 mm to (145.5, 133.0), turned to 90 degrees
- moved R28 165.7 mm to (141.0, 138.0), turned to 180 degrees
- moved R323 159.3 mm to (147.0, 138.0), turned to 180 degrees
- moved R322 147.5 mm to (160.0, 136.7), turned to 90 degrees
- moved R321 146.2 mm to (160.5, 133.0), turned to 90 degrees
- moved R205 145.1 mm to (113.5, 105.2), turned to 90 degrees
- moved R23 141.5 mm to (163.0, 133.0), turned to 90 degrees
- moved R58 141.4 mm to (186.8, 159.6), turned to 90 degrees
- moved R48 140.5 mm to (116.0, 105.2), turned to 90 degrees
- moved R41 139.6 mm to (118.5, 105.2), turned to 90 degrees
- moved R209 137.3 mm to (121.0, 105.2), turned to 90 degrees
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Connections:
- R25 pad 1: 3V3_AON -> (no net)
- R25 pad 2: Net-(J3-Pin_2) -> (no net)

Commit message: update
Parts:
- removed C61, C62, C63: DNP, Capacitor_SMD:C_0402_1005Metric
- removed R12, R49: DNP, Resistor_SMD:R_0603_1608Metric
- removed R47: 100k, Resistor_SMD:R_0603_1608Metric
- removed R50, R52: 10k, Resistor_SMD:R_0603_1608Metric
- removed R801: 10k, Resistor_SMD:R_0402_1005Metric
- C44: value 100nF -> 10nF
- C48: value 10uF 10V -> 4.7uF 10V
- L4: value 0.47uH 5.4A -> 0.47uH XGL4020-471MEC
- L5: value 2.2uH 4.4A -> 2.2uH XGL4020-222MEC
- moved J7 162.5 mm to (7.97, 2.52), turned to 0 degrees
- moved J6 161.6 mm to (2.58, 2.52), turned to 0 degrees
- moved R25 145.9 mm to (1.50, 8.80), turned to 0 degrees
- moved R38 137.6 mm to (129.3, 115.3), turned to 90 degrees
- moved R24 128.3 mm to (131.2, 115.3), turned to 90 degrees
- moved R22 128.2 mm to (133.2, 115.3), turned to 90 degrees
- moved R20 128.1 mm to (135.3, 115.3), turned to 90 degrees
- moved C52 122.9 mm to (137.0, 115.5), turned to 90 degrees
- moved D5 85.0 mm to (170.0, 104.3), turned to 0 degrees
- moved R68 77.5 mm to (96.4, 152.1)
- moved C76 62.7 mm to (170.5, 119.5)
- moved C77 59.3 mm to (150.8, 103.9)
- moved C78 56.6 mm to (166.0, 119.5)
- moved C79 56.6 mm to (167.5, 119.5)
- moved D7 56.4 mm to (170.5, 114.4), turned to 90 degrees
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Connections:
- R25 pad 1: (no net) -> 3V3_AON
- R25 pad 2: (no net) -> Net-(J3-Pin_2)
- U14 pad 1: Net-(U14-~{RESET}) -> Net-(J3-Pin_2)
- U19 pad 10: /MCU_PERIPHERALS/CAN1_TXD -> unconnected-(U19-CAN-TX+bootstrap(GPIO8)-Pad10)
- U19 pad 23: /MCU_PERIPHERALS/CAN1_RXD -> unconnected-(U19-CAN_RX+strap(GPIO15)-Pad23)
- U802 pad 3: /MCU_PERIPHERALS/TEMP_ALERT_N -> unconnected-(U802-ALERT-Pad3)

Commit message: update
Parts:
- moved C20 211.0 mm to (151.6, 155.9), turned to 90 degrees
- moved C23 199.4 mm to (135.3, 156.6)
- moved C18 196.7 mm to (144.8, 152.2)
- moved R25 188.4 mm to (138.7, 156.6)
- moved C16 188.3 mm to (135.3, 154.3)
- moved R21 184.2 mm to (138.7, 154.3)
- moved R20 181.7 mm to (144.8, 149.8)
- moved C22 181.6 mm to (144.8, 154.7)
- moved C64 134.8 mm to (138.8, 165.5)
- moved C66 133.1 mm to (138.8, 163.7)
- moved R75 63.8 mm to (119.7, 154.8), turned to 90 degrees
- moved R76 61.5 mm to (124.3, 154.7), turned to 90 degrees
- moved L3 45.1 mm to (148.9, 150.1)
- moved U7 37.6 mm to (140.6, 151.4)
- moved Q1 31.7 mm to (119.9, 163.7), turned to 180 degrees
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- renumbered SW2 to BOOT, C20 to C1, C22 to C10, C35 to C11, C21 to C12, C40 to C13, C36 to C14, C41 to C15, C45 to C16, C30 to C17, C43 to C18, C32 to C19, C42 to C2, C23 to C20, C24 to C21, C47 to C22, C46 to C23, C25 to C24, C6 to C25, C29 to C27, C7 to C28, C28 to C29, C33 to C3, C27 to C30, C8 to C31, C9 to C32, C5 to C33, C10 to C34, C11 to C35, C1 to C36, C13 to C37, C322 to C38, C14 to C39, C37 to C4, C2 to C40, C321 to C41, C323 to C42, C3 to C43, C12 to C44, C316 to C45, C18 to C46, C4 to C47, C15 to C48, C17 to C49, C38 to C5, C16 to C50, C44 to C51, C48 to C52, C49 to C53, C50 to C54, C51 to C55, C52 to C56, C53 to C57, C54 to C58, C55 to C59, C31 to C6, C56 to C60, C58 to C61, C57 to C62, C59 to C63, C60 to C64, C64 to C65, C65 to C66, C66 to C67, C67 to C68, C68 to C69, C19 to C7, C69 to C70, C70 to C71, C71 to C72, C72 to C73, C73 to C74, C312 to C75, C74 to C76, C313 to C77, C75 to C78, C76 to C79, C34 to C8, C77 to C80, C78 to C81, C79 to C82, C80 to C83, C81 to C84, C82 to C85, C83 to C86, C314 to C87, C84 to C88, C85 to C89, C39 to C9, C315 to C90, C86 to C91, C87 to C92, D2 to D1, D3 to D2, D1 to D3, J303 to J2, J2 to J3, J3 to J4, J4 to J5, J5 to J6, J6 to J7, J7 to J8, L5 to L1, L4 to L2, L8 to L3, L7 to L4, L3 to L5, L1 to L6, L301 to L7, L2 to L8, Q4 to Q1, Q5 to Q2, Q10 to Q3, Q2 to Q4, Q1 to Q5, R42 to R1, R36 to R10, R39 to R11, R29 to R12, R17 to R13, R18 to R14, R40 to R15, R31 to R16, R32 to R17, R21 to R18, R33 to R19, R43 to R2, R44 to R20, R46 to R21, R27 to R22, R26 to R23, R70 to R24, R45 to R25, R23 to R26, R322 to R27, R321 to R28, R323 to R29, R15 to R3, R28 to R30, R3 to R31, R4 to R32, R316 to R33, R7 to R34, R6 to R35, R10 to R36, R11 to R37, R313 to R38, R9 to R39, R16 to R4, R1 to R40, R2 to R41, R8 to R42, R601 to R43, R602 to R44, R202 to R45, R204 to R46, R203 to R47, R201 to R48, R25 to R49, R37 to R5, R20 to R50, R22 to R51, R24 to R52, R38 to R53, R34 to R54, R30 to R55, R906 to R56, R209 to R57, R205 to R58, R41 to R59, R13 to R6, R48 to R60, R51 to R61, R53 to R62, R55 to R63, R54 to R64, R56 to R65, R904 to R66, R57 to R67, R905 to R68, R58 to R69, R14 to R7, R59 to R70, R60 to R71, R61 to R72, R62 to R73, R63 to R74, R64 to R75, R65 to R76, R69 to R77, R66 to R78, R68 to R79, R19 to R8, R67 to R80, R35 to R9, SW1 to RESET, TP208 to TP1, TP311 to TP10, TP310 to TP11, TP309 to TP12, TP1 to TP13, TP7 to TP14, TP2 to TP15, TP205 to TP16, TP204 to TP17, TP14 to TP18, TP211 to TP19, TP3 to TP2, TP210 to TP20, TP201 to TP21, TP403 to TP22, TP12 to TP23, TP13 to TP24, TP15 to TP25, TP16 to TP26, TP17 to TP27, TP18 to TP28, TP19 to TP29, TP8 to TP3, TP20 to TP30, TP21 to TP31, TP22 to TP32, TP23 to TP33, TP24 to TP34, TP25 to TP35, TP9 to TP4, TP4 to TP5, TP10 to TP6, TP11 to TP7, TP6 to TP8, TP5 to TP9, U3 to U1, U2 to U10, U305 to U11, U1 to U12, U14 to U13, U12 to U14, U802 to U15, U15 to U16, U16 to U17, U17 to U18, U18 to U19, U8 to U2, U19 to U20, U20 to U21, U903 to U22, U902 to U23, U23 to U24, U24 to U25, U25 to U26, U26 to U27, U9 to U3, U6 to U4, U4 to U5, U7 to U6, U10 to U7, U11 to U8, U5 to U9

Commit message: udt
Parts:
- C35, CSC1, J1, J3: moved to B.Cu
- moved C13 206.2 mm to (188.8, 128.1)
- moved C9 204.5 mm to (188.8, 130.7)
- moved C4 203.8 mm to (188.9, 122.9)
- moved C15 203.5 mm to (188.8, 125.5)
- moved J7 169.3 mm to (102.1, 139.5), turned to 180 degrees
- moved R49 165.8 mm to (115.2, 129.4), turned to 90 degrees
- moved J8 162.0 mm to (102.1, 134.4), turned to 180 degrees
- moved R12 149.7 mm to (183.4, 130.4)
- moved R2 140.0 mm to (188.8, 120.7)
- moved C67 138.5 mm to (131.3, 159.7), turned to 90 degrees
- moved R11 130.9 mm to (183.4, 128.2)
- moved C68 130.1 mm to (135.1, 166.3)
- moved C69 127.6 mm to (135.1, 162.6)
- moved C70 127.6 mm to (135.1, 164.6)
- moved R15 126.4 mm to (183.4, 126.0)
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
Commit message: Update Tracker.kicad_pcb
Parts:
- moved C38 28.0 mm to (42.7, 81.3)
- moved C42 28.0 mm to (42.7, 83.3)
- moved C45 28.0 mm to (42.7, 79.3)
- moved C52 28.0 mm to (42.0, 88.0)
Changed lines of the file:
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@@
 	(footprint "Capacitor_SMD:C_0402_1005Metric"
 		(layer "F.Cu")
-		(at 23.6168 62.7482)
+		(at 42.7168 83.2582)
 		(descr "Capacitor SMD 0402 (1005 Metric), square (rectangular) end terminal, IPC-7351 nominal, (Body size source: IPC-SM-782 page 76, https://www.pcb-3d.com/wordpress/wp-content/uploads/ipc-sm-782a_amendment_1_and_2.pdf)")
 		(tags "capacitor")
@@
 	(footprint "Capacitor_SMD:C_0402_1005Metric"
 		(layer "F.Cu")
-		(at 23.6168 60.7782)
+		(at 42.7168 81.2882)
 		(descr "Capacitor SMD 0402 (1005 Metric), square (rectangular) end terminal, IPC-7351 nominal, (Body size source: IPC-SM-782 page 76, https://www.pcb-3d.com/wordpress/wp-content/uploads/ipc-sm-782a_amendment_1_and_2.pdf)")
 		(tags "capacitor")
@@
 	(footprint "Capacitor_SMD:C_0805_2012Metric"
 		(layer "F.Cu")
-		(at 22.95 67.49)
+		(at 42.05 88)
 		(descr "Capacitor SMD 0805 (2012 Metric), square (rectangular) end terminal, IPC-7351 nominal, (Body size source: IPC-SM-782 page 76, https://www.pcb-3d.com/wordpress/wp-content/uploads/ipc-sm-782a_amendment_1_and_2.pdf, https://docs.google.com/spreadsheets/d/1BsfQQcO9C6DZCsRaXUlFlo91Tg2WpOkGARC1WS5S8t0/edit?usp=sharing)")
 		(tags "capacitor")
@@
 	(footprint "Capacitor_SMD:C_0402_1005Metric"
 		(layer "F.Cu")
-		(at 23.6168 58.8082)
+		(at 42.7168 79.3182)
 		(descr "Capacitor SMD 0402 (1005 Metric), square (rectangular) end terminal, IPC-7351 nominal, (Body size source: IPC-SM-782 page 76, https://www.pcb-3d.com/wordpress/wp-content/uploads/ipc-sm-782a_amendment_1_and_2.pdf)")
 		(tags "capacitor")

Commit message: BT1 update
Parts:
- BT1: footprint SamacSys_Parts:BHC186501P -> Battery:BatteryHolder_MPD_BH-18650-PC
- J4: moved to B.Cu
- moved CSC1 0.43 mm to (169.7, 133.6)
- turned J4 to 0 degrees
- renumbered BOOT to BOOT1, RESET to RESET1
