File: Tracker.kicad_pcb (KiCad board)
At the start: 4 copper layers, 100 x 70 mm, 277 parts, among them J1 Vehicle 12V 2X2, J2 Conn_Coaxial, J3 USB_C_Receptacle_USB2.0_16P, J4 Conn_01x05, J5 Micro_SD_Card_Det_Hirose_DM3AT, J6 SIM8060-6-1-14-00-A, J7 Conn_Coaxial, J8 Conn_Coaxial, Q1 CSD16406Q3, Q2 CSD16406Q3, Q3 2N7002, Q4 2N7002, Q5 DMT6007LFGQ-7, Q6 MMBT3904, Q7 MMBT3904, U1 TPS2121RUXR, U10 LM76003QRNPRQ1, U11 MAX-M10S, U12 LM74700, U13 TPS3840DL30DBVR, U14 USBLC6-2SC6, U15 TMP1075DGKR, U16 ATECC608B-SSHDA, U17 USBLC6-2SC6, U18 ASM330LHHTR, U19 TCA9535PWR, U2 TPS63802DLAR, U21 W25N01GVZEIG, U22 SN74AXC4T245QPWRQ1, U23 SN74AXC4T245QPWRQ1, U24 TPS22918TDBVTQ1, U25 SN74AXC4T245QPWRQ1_CELL, U26 SN74AXC4T245QPWRQ1, U27 BG95-M3, U3 TPS61094DSSR, U4 BQ29700DSER, U5 INA3221AIRGVR, U6 TPS3840DL35DBVR, U7 TPS62840DLCR, U8 TPS62840DLCR, U9 BQ25601DRTWR

Commit message: Fix
Parts:
- removed BT1: BHC-18650-1P, Battery:BatteryHolder_MPD_BH-18650-PC
- added BT2: BH-18650-PC, Battery:BatteryHolder_MPD_BH-18650-PC, B.Cu at (188.9, 158.5)
- added TP36: ~, TestPoint:TestPoint_Pad_D1.5mm, B.Cu at (140.9, 110.5)
- C54: value 100nF -> 10uF
- C63: value 10nF -> 100nF
- L8, TH1: moved to B.Cu
- moved TH1 33.2 mm to (138.3, 146.0), turned to 0 degrees
- moved R57 30.2 mm to (116.5, 131.9)
- moved C51 27.3 mm to (134.8, 132.8), turned to 0 degrees
- moved R59 26.7 mm to (118.4, 131.9)
- moved R55 25.8 mm to (115.8, 108.3), turned to -90 degrees
- moved R45 25.3 mm to (107.9, 108.2)
- moved L8 18.9 mm to (185.9, 143.2), turned to 0 degrees
- moved R34 14.3 mm to (178.3, 135.3), turned to -90 degrees
- moved C48 11.1 mm to (176.0, 144.9), turned to -90 degrees
- moved C62 10.2 mm to (124.1, 139.0), turned to -90 degrees
- moved TP14 10.2 mm to (177.8, 145.8)
- moved R35 9.98 mm to (181.3, 145.0), turned to 90 degrees
- moved C42 9.46 mm to (118.5, 140.3)
- moved R39 9.16 mm to (179.5, 144.9), turned to 90 degrees
- moved R49 9.08 mm to (109.8, 131.7)
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Connections:
- C35 pad 1: GND -> Net-(U10-PVIN_1)
- C35 pad 2: Net-(U10-PVIN_1) -> GND
