File: Tracker.kicad_pcb (KiCad board)
At the start: 4 copper layers, 100 x 70 mm, 278 parts, among them J1 Vehicle 12V 2X2, J2 Conn_Coaxial, J3 USB_C_Receptacle_USB2.0_16P, J4 Conn_01x05, J5 Micro_SD_Card_Det_Hirose_DM3AT, J6 SIM8060-6-1-14-00-A, J7 Conn_Coaxial, J8 Conn_Coaxial, Q1 CSD16406Q3, Q2 CSD16406Q3, Q3 2N7002, Q4 2N7002, Q5 DMT6007LFGQ-7, Q6 MMBT3904, Q7 MMBT3904, U1 TPS2121RUXR, U10 LM76003QRNPRQ1, U11 MAX-M10S, U12 LM74700, U13 TPS3840DL30DBVR, U14 USBLC6-2SC6, U15 TMP1075DGKR, U16 ATECC608B-SSHDA, U17 USBLC6-2SC6, U18 ASM330LHHTR, U19 TCA9535PWR, U2 TPS63802DLAR, U21 W25N01GVZEIG, U22 SN74AXC4T245QPWRQ1, U23 SN74AXC4T245QPWRQ1, U24 TPS22918TDBVTQ1, U25 SN74AXC4T245QPWRQ1_CELL, U26 SN74AXC4T245QPWRQ1, U27 BG95-M3, U3 TPS61094DSSR, U4 BQ29700DSER, U5 INA3221AIRGVR, U6 TPS3840DL35DBVR, U7 TPS62840DLCR, U8 TPS62840DLCR, U9 BQ25601DRTWR

Commit message: updt
Parts:
- moved C52 16.8 mm to (185.7, 107.0)
- moved D3 16.7 mm to (189.9, 104.1)
- moved F2 16.6 mm to (189.9, 106.8)
- moved TP4 8.48 mm to (180.6, 110.2)
- moved C66 7.68 mm to (142.5, 156.9)
- moved R20 7.42 mm to (142.4, 152.8), turned to -90 degrees
- moved C18 6.44 mm to (139.5, 148.5), turned to 90 degrees
- moved C22 4.80 mm to (145.0, 150.5), turned to -90 degrees
- moved C17 3.43 mm to (150.7, 149.1)
- moved L3 1.86 mm to (142.7, 150.0), turned to 90 degrees
- moved C64 1.74 mm to (140.4, 164.8)
- moved C54 0.58 mm to (134.3, 141.6)
- moved C55 0.58 mm to (134.3, 143.0)
- moved C58 0.58 mm to (134.3, 144.4)
Changed lines of the file:
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@@
 		(capping no)
 		(filling no)
+		(zone_defaults)
 		(pcbplotparams
 			(layerselection 0x00000000_00000000_55555555_5755f5ff)
@@
 	(footprint "Capacitor_SMD:C_0603_1608Metric"
 		(layer "F.Cu")
-		(at 149.25 152.25 180)
+		(at 150.675 149.125 180)
 		(descr "Capacitor SMD 0603 (1608 Metric), square (rectangular) end terminal, IPC-7351 nominal, (Body size source: IPC-SM-782 page 76, https://www.pcb-3d.com/wordpress/wp-content/uploads/ipc-sm-782a_amendment_1_and_2.pdf)")
 		(tags "capacitor")
@@
 	(footprint "Capacitor_SMD:C_0402_1005Metric"
 		(layer "F.Cu")
-		(at 138.8 165.5)
+		(at 140.38 164.775)
 		(descr "Capacitor SMD 0402 (1005 Metric), square (rectangular) end terminal, IPC-7351 nominal, (Body size source: IPC-SM-782 page 76, https://www.pcb-3d.com/wordpress/wp-content/uploads/ipc-sm-782a_amendment_1_and_2.pdf)")
 		(tags "capacitor")
@@
 	(footprint "Capacitor_SMD:C_0805_2012Metric"
 		(layer "F.Cu")
-		(at 146.25 155.1 90)
+		(at 144.975 150.475 -90)
 		(descr "Capacitor SMD 0805 (2012 Metric), square (rectangular) end terminal, IPC-7351 nominal, (Body size source: IPC-SM-782 page 76, https://www.pcb-3d.com/wordpress/wp-content/uploads/ipc-sm-782a_amendment_1_and_2.pdf, https://docs.google.com/spreadsheets/d/1BsfQQcO9C6DZCsRaXUlFlo91Tg2WpOkGARC1WS5S8t0/edit?usp=sharing)")
 		(tags "capacitor")
@@
 		(duplicate_pad_numbers_are_jumpers no)
 		(fp_line
-			(start -0.261252 -0.735)
-			(end 0.261252 -0.735)
+			(start -0.261252 0.735)
+			(end 0.261252 0.735)
 			(stroke
 				(width 0.12)
@@
 		)
 		(fp_line
-			(start -0.261252 0.735)
-			(end 0.261252 0.735)
+			(start -0.261252 -0.735)
+			(end 0.261252 -0.735)
 			(stroke
 				(width 0.12)
@@
 		)
 		(pad "1" smd roundrect
-			(at -0.95 0 90)
+			(at -0.95 0 270)
 			(size 1 1.45)
 			(layers "F.Cu" "F.Mask" "F.Paste")
@@
 		)
 		(pad "2" smd roundrect
-			(at 0.95 0 90)
+			(at 0.95 0 270)
 			(size 1 1.45)
 			(layers "F.Cu" "F.Mask" "F.Paste")
@@
 	(footprint "Capacitor_SMD:C_0402_1005Metric"
 		(layer "F.Cu")
-		(at 134.875 144.525)
+		(at 134.305 144.4)
 		(descr "Capacitor SMD 0402 (1005 Metric), square (rectangular) end terminal, IPC-7351 nominal, (Body size source: IPC-SM-782 page 76, https://www.pcb-3d.com/wordpress/wp-content/uploads/ipc-sm-782a_amendment_1_and_2.pdf)")
 		(tags "capacitor")
@@
 	(footprint "Inductor_SMD:L_Murata_DFE201610P"
 		(layer "F.Cu")
-		(at 144.5 149.55)
+		(at 142.7 150.025 90)
 		(descr "Inductor, Murata, DFE201610P, 2.0x1.6x1.0mm, (https://www.murata.com/~/media/webrenewal/products/inductor/chip/tokoproducts/wirewoundmetalalloychiptype/m_dfe201610p.ashx)")
 		(tags "power chip flatwire")
 		(property "Reference" "L3"
-			(at 0 -1.75 0)
+			(at 0 -1.75 90)
 			(layer "F.SilkS")
 			(effects
@@
 		)
 		(property "Value" "2.2uH"
-			(at 0 1.75 0)
+			(at 0 1.75 90)
 			(layer "F.Fab")
 			(effects
@@
 		)
 		(property "Datasheet" ""
-			(at 0 0 0)
+			(at 0 0 90)
 			(layer "F.Fab")
 			(hide yes)
@@
 		)
 		(property "Description" "Inductor"
-			(at 0 0 0)
+			(at 0 0 90)
 			(layer "F.Fab")
 			(hide yes)
@@
 		)
 		(property "KiLib_Generator" "inductor/SMD"
-			(at 0 0 0)
+			(at 0 0 90)
 			(layer "F.SilkS")
 			(hide yes)
@@
 		)
 		(fp_text user "${REFERENCE}"
-			(at 0 0 0)
+			(at 0 0 90)
 			(layer "F.Fab")
 			(effects
@@
 		)
 		(pad "1" smd roundrect
-			(at -0.725 0)
+			(at -0.725 0 90)
 			(size 0.55 1.6)
 			(layers "F.Cu" "F.Mask" "F.Paste")
@@
 		)
 		(pad "2" smd roundrect
-			(at 0.725 0)
+			(at 0.725 0 90)
 			(size 0.55 1.6)
 			(layers "F.Cu" "F.Mask" "F.Paste")
@@
 	(footprint "Capacitor_SMD:C_0402_1005Metric"
 		(layer "F.Cu")
-		(at 138.82 163.7)
+		(at 142.475 156.95)
 		(descr "Capacitor SMD 0402 (1005 Metric), square (rectangular) end terminal, IPC-7351 nominal, (Body size source: IPC-SM-782 page 76, https://www.pcb-3d.com/wordpress/wp-content/uploads/ipc-sm-782a_amendment_1_and_2.pdf)")
 		(tags "capacitor")
@@
 	(footprint "Resistor_SMD:R_0603_1608Metric"
 		(layer "F.Cu")
-		(at 149.125 149.7)
+		(at 142.4 152.825 -90)
 		(descr "Resistor SMD 0603 (1608 Metric), square (rectangular) end terminal, IPC-7351 nominal, (Body size source: IPC-SM-782 page 72, https://www.pcb-3d.com/wordpress/wp-content/uploads/ipc-sm-782a_amendment_1_and_2.pdf)")
 		(tags "resistor")
 		(property "Reference" "R20"
-			(at -0.025 -1.2 0)
+			(at -0.025 -1.2 90)
 			(layer "F.SilkS")
 			(effects
@@
 		)
 		(property "Value" "267k 1%"
-			(at 0 1.43 0)
+			(at 0 1.43 90)
 			(layer "F.Fab")
 			(effects
@@
 		)
 		(property "Datasheet" ""
-			(at 0 0 0)
+			(at 0 0 90)
 			(layer "F.Fab")
 			(hide yes)
@@
 		)
 		(property "Description" "Resistor"
-			(at 0 0 0)
+			(at 0 0 90)
 			(layer "F.Fab")
 			(hide yes)
@@
 		)
 		(property "KiLib_Generator" "SMD_2terminal_chip_molded"
-			(at 0 0 0)
+			(at 0 0 90)
 			(layer "F.SilkS")
 			(hide yes)
@@
 		(duplicate_pad_numbers_are_jumpers no)
 		(fp_line
-			(start -0.237258 -0.5225)
-			(end 0.237258 -0.5225)
+			(start -0.237258 0.5225)
+			(end 0.237258 0.5225)
 			(stroke
 				(width 0.12)
@@
 		)
 		(fp_line
-			(start -0.237258 0.5225)
-			(end 0.237258 0.5225)
+			(start -0.237258 -0.5225)
+			(end 0.237258 -0.5225)
 			(stroke
 				(width 0.12)
@@
 		)
 		(fp_text user "${REFERENCE}"
-			(at 0 0 0)
+			(at 0 0 90)
 			(layer "F.Fab")
 			(effects
@@
 		)
 		(pad "1" smd roundrect
-			(at -0.825 0)
+			(at -0.825 0 270)
 			(size 0.8 0.95)
 			(layers "F.Cu" "F.Mask" "F.Paste")
@@
 		)
 		(pad "2" smd roundrect
-			(at 0.825 0)
+			(at 0.825 0 270)
 			(size 0.8 0.95)
 			(layers "F.Cu" "F.Mask" "F.Paste")
@@
 	(footprint "Capacitor_SMD:C_0402_1005Metric"
 		(layer "F.Cu")
-		(at 134.88 141.75)
+		(at 134.31 141.625)
 		(descr "Capacitor SMD 0402 (1005 Metric), square (rectangular) end terminal, IPC-7351 nominal, (Body size source: IPC-SM-782 page 76, https://www.pcb-3d.com/wordpress/wp-content/uploads/ipc-sm-782a_amendment_1_and_2.pdf)")
 		(tags "capacitor")
@@
 		)
 		(embedded_fonts no)
-		(model "${KICAD10_3DMODEL_DIR}/Capacitor_SMD.3dshapes/C_0402_1005Metric.step"
+		(model "${KICAD10_3DMODEL_DIR}/Capacitor_SMD.3dshapes/C_0603_1608Metric.step"
 			(offset
 				(xyz 0 0 0)
@@
 	(footprint "Capacitor_SMD:C_0402_1005Metric"
 		(layer "F.Cu")
-		(at 134.875 143.125)
+		(at 134.305 143)
 		(descr "Capacitor SMD 0402 (1005 Metric), square (rectangular) end terminal, IPC-7351 nominal, (Body size source: IPC-SM-782 page 76, https://www.pcb-3d.com/wordpress/wp-content/uploads/ipc-sm-782a_amendment_1_and_2.pdf)")
 		(tags "capacitor")
@@
 	(footprint "Capacitor_SMD:C_0603_1608Metric"
 		(layer "F.Cu")
-		(at 144.775 152.2)
+		(at 139.5 148.5 90)
 		(descr "Capacitor SMD 0603 (1608 Metric), square (rectangular) end terminal, IPC-7351 nominal, (Body size source: IPC-SM-782 page 76, https://www.pcb-3d.com/wordpress/wp-content/uploads/ipc-sm-782a_amendment_1_and_2.pdf)")
 		(tags "capacitor")
 		(property "Reference" "C18"
-			(at -0.075 -1.2 0)
+			(at -0.075 -1.2 90)
 			(layer "F.SilkS")
 			(effects
@@
 		)
 		(property "Value" "4.7uF 10V"
-			(at 0 1.43 0)
+			(at 0 1.43 90)
 			(layer "F.Fab")
 			(effects
@@
 		)
 		(property "Datasheet" ""
-			(at 0 0 0)
+			(at 0 0 90)
 			(layer "F.Fab")
 			(hide yes)
@@
 		)
 		(property "Description" "Unpolarized capacitor"
-			(at 0 0 0)
+			(at 0 0 90)
 			(layer "F.Fab")
 			(hide yes)
@@
 		)
 		(property "KiLib_Generator" "SMD_2terminal_chip_molded"
-			(at 0 0 0)
+			(at 0 0 90)
 			(layer "F.SilkS")
 			(hide yes)
@@
 		)
 		(fp_text user "${REFERENCE}"
-			(at 0 0 0)
+			(at 0 0 90)
 			(layer "F.Fab")
 			(effects
@@
 		)
 		(pad "1" smd roundrect
-			(at -0.775 0)
+			(at -0.775 0 90)
 			(size 0.9 0.95)
 			(layers "F.Cu" "F.Mask" "F.Paste")
@@
 		)
 		(pad "2" smd roundrect
-			(at 0.775 0)
+			(at 0.775 0 90)
 			(size 0.9 0.95)
 			(layers "F.Cu" "F.Mask" "F.Paste")
@@
 	(footprint "Diode_SMD:D_SMF"
 		(layer "B.Cu")
-		(at 192.925 120.5)
+		(at 189.875 104.1)
 		(descr "Diode SMF (DO-219AB), http://www.vishay.com/docs/95572/smf_do-219ab.pdf")
 		(tags "Diode SMF (DO-214AB)")
@@
 	(footprint "TestPoint:TestPoint_Pad_D1.5mm"
 		(layer "B.Cu")
-		(at 188.375 106.85 -90)
+		(at 180.6 110.225 -90)
 		(descr "SMD pad as test Point, diameter 1.5mm")
 		(tags "test point SMD pad")
@@
 	(footprint "Capacitor_SMD:C_0805_2012Metric"
 		(layer "B.Cu")
-		(at 188.15 123.65 180)
+		(at 185.725 107.025 180)
 		(descr "Capacitor SMD 0805 (2012 Metric), square (rectangular) end terminal, IPC-7351 nominal, (Body size source: IPC-SM-782 page 76, https://www.pcb-3d.com/wordpress/wp-content/uploads/ipc-sm-782a_amendment_1_and_2.pdf, https://docs.google.com/spreadsheets/d/1BsfQQcO9C6DZCsRaXUlFlo91Tg2WpOkGARC1WS5S8t0/edit?usp=sharing)")
 		(tags "capacitor")
@@
 			)
 		)
-		(attr through_hole)
+		(attr through_hole dnp)
 		(duplicate_pad_numbers_are_jumpers no)
 		(fp_line
@@
 		)
 		(embedded_fonts no)
-		(model "${KICAD10_3DMODEL_DIR}/Battery.3dshapes/BatteryHolder_MPD_BH-18650-PC.step"
+		(model "${KICAD10_3DMODEL_DIR}/Battery.3dshapes/BatteryHolder_MPD_BH-18650-PC2.step"
 			(offset
 				(xyz 0 0 0)
@@
 	(footprint "Fuse:Fuse_1206_3216Metric"
 		(layer "B.Cu")
-		(at 192.85 123.175 180)
+		(at 189.925 106.825 180)
 		(descr "Fuse SMD 1206 (3216 Metric), square (rectangular) end terminal, IPC-7351 nominal, (Body size source: http://www.tortai-tech.com/upload/download/2011102023233369053.pdf)")
 		(tags "fuse")

Commit message: updt
Parts:
- removed REF** (x4): MountingHole_3.2mm_M3, MountingHole:MountingHole_3.2mm_M3
- added H1: MountingHole_3.2mm_M3, MountingHole:MountingHole_3.2mm_M3, F.Cu at (104.0, 104.0)
- added H2: MountingHole_3.2mm_M3, MountingHole:MountingHole_3.2mm_M3, F.Cu at (104.0, 166.0)
- added H3: MountingHole_3.2mm_M3, MountingHole:MountingHole_3.2mm_M3, F.Cu at (196.0, 104.0)
- added H4: MountingHole_3.2mm_M3, MountingHole:MountingHole_3.2mm_M3, F.Cu at (196.0, 166.0)
- BT2: footprint Battery:BatteryHolder_MPD_BH-18650-PC -> SamacSys_Parts:BAT_BH-18650-PC
- moved BT2 39.5 mm to (149.5, 157.9)
- moved C72 11.3 mm to (126.1, 124.1)
- moved R72 2.66 mm to (131.5, 124.2)
- moved R70 2.49 mm to (128.8, 124.2)
- moved R73 0.75 mm to (134.7, 123.3)
- moved R71 0.63 mm to (134.8, 122.0)
- moved C74 0.63 mm to (134.8, 120.8)

Commit message: Update Tracker.kicad_pcb
Parts:
- moved C25 13.9 mm to (168.1, 128.0), turned to 180 degrees
- moved J7 11.3 mm to (140.3, 102.0)
- moved C28 10.2 mm to (168.1, 131.4), turned to 180 degrees
- moved C77 9.52 mm to (160.1, 103.2), turned to 90 degrees
- moved C32 8.53 mm to (180.0, 130.6), turned to 90 degrees
- moved C75 8.35 mm to (161.5, 103.2), turned to 90 degrees
- moved C8 8.31 mm to (172.1, 120.8), turned to -90 degrees
- moved C34 8.18 mm to (177.4, 131.4), turned to -90 degrees
- moved C11 8.08 mm to (172.2, 124.5), turned to 90 degrees
- moved R10 7.32 mm to (164.8, 123.5)
- moved R9 7.29 mm to (164.8, 126.5)
- moved R77 6.25 mm to (158.5, 104.2), turned to 90 degrees
- moved R80 5.78 mm to (142.7, 104.6), turned to 180 degrees
- moved C31 5.52 mm to (172.5, 134.5), turned to 0 degrees
- moved C92 5.50 mm to (160.7, 127.6)
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