File: cellular.kicad_sch (KiCad schematic)
At the start: 54 parts, among them J5 SIM8060-6-1-14-00-A, J6 Conn_Coaxial, J7 Conn_Coaxial, Q6 MMBT3904, Q7 MMBT3904, U24 SN74AXC4T245QPWRQ1, U25 SN74AXC4T245QPWRQ1, U26 BG95-M3

Commit message: Bug fix
Parts:
- J5: symbol SamacSys_Parts:SIM8060-6-1-14-00-A -> Project_Parts:SIM8060-6-1-14-00-A
- Q6, Q7: symbol SamacSys_Parts:MMBT3904 -> Project_Parts:MMBT3904
- U24: value SN74AXC4T245QPWRQ1 -> SN74AXC4T245QPWRQ1_CELL; symbol SamacSys_Parts:SN74AXC4T245QPWRQ1 -> Project_Parts:SN74AXC4T245QPWRQ1_CELL; now left out of the parts list
- U26: symbol RF_GSM:BG95-M3 -> Project_Parts:BG95-M3

Commit message: update
Parts:
- renumbered C70 to C71, C71 to C72, C72 to C73, C73 to C74, C312 to C75, C74 to C76, C313 to C77, C75 to C78, C76 to C79, C77 to C80, C78 to C81, C79 to C82, C80 to C83, C81 to C84, C82 to C85, C83 to C86, C314 to C87, C84 to C88, C85 to C89, C315 to C90, C86 to C91, C87 to C92, J5 to J6, J6 to J7, J7 to J8, R59 to R70, R60 to R71, R61 to R72, R62 to R73, R63 to R74, R64 to R75, R65 to R76, R69 to R77, R66 to R78, R68 to R79, R67 to R80, TP18 to TP28, TP19 to TP29, TP20 to TP30, TP21 to TP31, TP22 to TP32, TP23 to TP33, TP24 to TP34, TP25 to TP35, U24 to U25, U25 to U26, U26 to U27

Commit message: Fix
Parts:
- added TP36: (no value), TestPoint:TestPoint_Pad_D1.5mm, symbol Connector:TestPoint
Connections:
- net GND: now also TP36.1
Changed lines of the file:
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@@
+	)
+	(symbol
+		(lib_id "Connector:TestPoint")
+		(at 133.35 151.13 90)
+		(unit 1)
+		(body_style 1)
+		(exclude_from_sim no)
+		(in_bom yes)
+		(on_board yes)
+		(in_pos_files yes)
+		(dnp no)
+		(property "Reference" "TP36"
+			(at 126.238 151.384 90)
+			(show_name no)
+			(do_not_autoplace no)
+			(effects
+				(font
+					(size 1.27 1.27)
+				)
+			)
+		)
+		(property "Value" ""
+			(at 130.048 148.59 90)
+			(show_name no)
+			(do_not_autoplace no)
+			(effects
+				(font
+					(size 1.27 1.27)
+				)
+			)
+		)
+		(property "Footprint" "TestPoint:TestPoint_Pad_D1.5mm"
+			(at 133.35 146.05 0)
+			(hide yes)
+			(show_name no)
+			(do_not_autoplace no)
+			(effects
+				(font
+					(size 1.27 1.27)
+				)
+			)
+		)
+		(property "Datasheet" ""
+			(at 133.35 146.05 0)
+			(hide yes)
+			(show_name no)
+			(do_not_autoplace no)
+			(effects
+				(font
+					(size 1.27 1.27)
+				)
+			)
+		)
+		(property "Description" "test point"
+			(at 133.35 151.13 0)
+			(hide yes)
+			(show_name no)
+			(do_not_autoplace no)
+			(effects
+				(font
+					(size 1.27 1.27)
+				)
+			)
+		)
+		(pin "1"
+		)
+		(instances
+			(project "Tracker"
+				(path "/586d1ea1-b017-4713-987c-545d658f6cc8/14966949-e78d-448f-9d65-c3e7a44dd897"
+					(reference "TP36")
+					(unit 1)
+				)
+			)
+		)
 	)
 	(symbol
